File: pcb/hv.kicad_sch (KiCad schematic)
At the start: 32 parts, among them Q201 IRL540N, T201 DA2032-AL, U201 LM5155

Commit message: Add title and revision to schematic and board silkscreen, do a bit of tidying of the schematics
Other:
- note added: "170V Flyback Converter"
- title: (none) -> ${TITLE}
Changed lines of the file:
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@@
 	(generator_version "9.0")
 	(paper "A4")
+	(title_block
+		(title "${TITLE}")
+		(rev "${REV}")
+	)
+	(rectangle
+		(start 59.69 57.15)
+		(end 227.33 149.86)
+		(stroke
+			(width 0)
+			(type default)
+		)
+		(fill
+			(type none)
+		)
+	)
+	(text "170V Flyback Converter"
+		(exclude_from_sim no)
+		(at 59.69 56.388 0)
+		(effects
+			(font
+				(size 1.27 1.27)
+			)
+			(justify left)
+		)
+	)
 	(junction
 		(at 151.13 69.85)

Commit message: Add ESP32, finish wiring. Rev A complete
Parts:
- T201: MFG Part No (none) -> DA2032-AL
- U201: MFG Part No (none) -> LM51551DSSR
Connections:
- net PGOOD renamed PGOOD_{LM5155}
Changed lines of the file:
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@@
-		)
-	)
-	(label "PGOOD"
-		(at 76.2 111.76 0)
-		(effects
-			(font
-				(size 1.27 1.27)
-			)
-			(justify left bottom)
 		)
 	)
@@
 		)
 	)
+	(global_label "PGOOD_{LM5155}"
+		(shape output)
+		(at 76.2 111.76 180)
+		(fields_autoplaced yes)
+		(effects
+			(font
+				(size 1.27 1.27)
+			)
+			(justify right)
+		)
+		(property "Intersheetrefs" "${INTERSHEET_REFS}"
+			(at 60.839 111.76 0)
+			(effects
+				(font
+					(size 1.27 1.27)
+				)
+				(justify right)
+				(hide yes)
+			)
+		)
+	)
 	(symbol
 		(lib_id "power:GND")
@@
 			)
 		)
-		(property "MFG Part No" ""
+		(property "MFG Part No" "LM51551DSSR"
 			(at 114.3 109.22 0)
 			(effects
@@
 			)
 		)
-		(property "MFG Part No" ""
+		(property "MFG Part No" "DA2032-AL"
 			(at 165.1 76.2 0)
 			(effects

Commit message: Partial Rev B, committing before splitting projects
Parts:
- removed C211: 1uF, nixie_clock:C_Rect_L7.1mm_W4.1mm_P5.08mm_Goldmax, symbol Device:C
- added C109: 10nF, nixie_clock:C_Rect_L5.1mm_W3.2mm_P5.08mm_Goldmax, symbol Device:C
- added D1: SB240S, Diode_THT:D_DO-41_SOD81_P7.62mm_Horizontal, symbol Device:D
- added H6, H7, H8, H9: MountingHole, MountingHole:MountingHole_3.2mm_M3_ISO7380, symbol Mechanical:MountingHole
- added Q151: TN2106N3-G, Package_TO_SOT_THT:TO-92L, symbol Transistor_FET:Q_NMOS_SGD
- added R13: 3.3, Resistor_THT:R_Axial_DIN0207_L6.3mm_D2.5mm_P7.62mm_Horizontal, symbol Device:R
- added R160: 100k, Resistor_THT:R_Axial_DIN0207_L6.3mm_D2.5mm_P7.62mm_Horizontal, symbol Device:R
- C13: renamed from C209; value 10nF -> 12nF; MFG Part No C317C103K1R5TA7301 -> C317C123K1R5TA7301
- C9: renamed from C206; value 47nF -> 220nF; MFG Part No C322C473J5R5TA -> C322C224K5R5TA7301
- R12: renamed from R212; value 27k -> 30k; MFG Part No MFR-25FRF52-27K -> MFR-25FRF52-30K
- R20: renamed from R202; value 470k -> 1.5M; MFG Part No MFR-25FRF52-470K -> MFR-25FBF52-1M5
- U5: renamed from U201; footprint Package_SON:WSON-12-1EP_3x2mm_P0.5mm_EP1x2.65_ThermalVias -> nixie_clock:WSON-12-1EP_3x2mm_P0.5mm_EP1x2.65_ThermalVias
- renumbered C207 to C10, C210 to C11, C208 to C12, C204 to C14, C205 to C15, C202 to C5, C203 to C6, C201 to C7, D202 to D2, D201 to D3, Q201 to Q1, R209 to R10, R210 to R11, R211 to R14, R213 to R15, R201 to R16, R203 to R17, R204 to R18, R205 to R19, R206 to R7, R207 to R8, R208 to R9, RV201 to RV1, T201 to T1, TP202 to TP1, TP201 to TP2
Connections:
- net +3V3: now also R160.1
- net GND: now also C109.1, Q151.1 (S)
- net UVLO: now also Q151.3 (D)
- net V_{BUS}: now also C109.2
- net GATE_{IRL540N}: now reaches Q1.1 (G), R14.2
- net GATE_{IRL540N}: now also R13.2
- net SOURCE_{IRL540N}: now reaches Q1.3 (S), R15.1, R16.1
- net GATE renamed GATE_{LM5155}
- net GATE_{LM5155}: now also D1.1 (K)
- new net: D1.2 (A), R13.1
- new net EN_{HV}: Q151.2 (G), R160.2
Other:
- moved on the sheet: R14, R7
