File: pcb/main/main.kicad_pcb (KiCad board)
At the start: 2 copper layers, 70 x 65 mm, 96 parts, among them J101 USB_C_Receptacle_USB2.0_16P, J102 Conn_01x06, J103 Conn_02x13_Counter_Clockwise, J151 UART, J152 JTAG, Q101 Q_Dual_PMOS_S1G1S2G2D2D2D1D1, Q121 PMF170XP, SW151 Boot, SW152 Reset, U101 USBLC6-2SC6, U102 TS3USB221A, U103 CYPD3176, U121 TPS63070, U131 TPS629203, U151 74LVC1G17, U152 74LVC1G17, U153 ESP32-S3-WROOM-1

Commit message: Rev B RC1
Parts:
- removed H101, H102, H103, H104: MountingHole, MountingHole:MountingHole_3.2mm_M3_ISO7380
- removed J152: JTAG, Connector_PinHeader_2.54mm:PinHeader_1x04_P2.54mm_Vertical
- added H2: MountingHole, MountingHole:MountingHole_3.2mm_M3_ISO7380, F.Cu at (105.0, 60.0)
- added H3: MountingHole, MountingHole:MountingHole_3.2mm_M3_ISO7380, F.Cu at (165.0, 60.0)
- added H4: MountingHole, MountingHole:MountingHole_3.2mm_M3_ISO7380, F.Cu at (105.0, 115.0)
- added H5: MountingHole, MountingHole:MountingHole_3.2mm_M3_ISO7380, F.Cu at (165.0, 115.0)
- added J2: JTAG, nixie_clock:Samtec_FTSH-105-01-L-DV-K_2x05_P1.27mm_Vertical_SMD, F.Cu at (112.5, 112.0)
- added J3: JTAG SRC, Connector_PinHeader_2.54mm:PinHeader_1x02_P2.54mm_Vertical, F.Cu at (149.0, 91.5)
- added R6: 100k, Resistor_SMD:R_0402_1005Metric, F.Cu at (146.0, 94.8)
- added R7: 10k, Resistor_SMD:R_0402_1005Metric, F.Cu at (146.0, 93.8)
- D3: renamed from D153; value HB -> STATUS
- J4: renamed from J103; value Conn_02x13_Counter_Clockwise -> 26 pin IDC
- moved D3 43.6 mm to (111.5, 89.0)
- moved R8 43.6 mm to (110.1, 88.8)
- moved R10 24.7 mm to (122.6, 98.5), turned to 90 degrees
- moved D1 11.2 mm to (109.0, 103.7)
- moved D2 11.2 mm to (109.0, 102.0)
- moved R3 11.2 mm to (108.5, 105.0)
- moved R4 11.2 mm to (108.5, 100.7)
- moved J1 11.1 mm to (103.4, 94.2)
- moved C2 7.05 mm to (117.9, 100.8)
- moved R2 7.05 mm to (112.6, 101.1)
- moved U1 7.05 mm to (115.2, 104.5)
- moved U2 7.05 mm to (115.2, 101.1)
- moved C1 7.05 mm to (114.1, 106.7)
- moved R1 7.05 mm to (112.6, 103.0)
- moved R5 7.05 mm to (117.8, 105.0)
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- renumbered C151 to C1, C152 to C2, C153 to C3, C154 to C4, C155 to C5, D151 to D1, D152 to D2, J151 to J1, J102 to J5, R151 to R1, R159 to R10, R158 to R11, R152 to R2, R153 to R3, R154 to R4, R155 to R5, R157 to R8, R156 to R9, SW151 to SW1, SW152 to SW2, TP151 to TP1, U151 to U1, U152 to U2, U153 to U3
Connections:
- net /MCU/BOOT renamed /mcu/BOOT
- net /MCU/RXD0 renamed /mcu/RXD0
- net /MCU/RXD0_{B} renamed /mcu/RXD0_{B}
- net /MCU/TXD0 renamed /mcu/TXD0
- net /MCU/TXD0_{B0} renamed /mcu/TXD0_{B0}
- net /MCU/TXD0_{B1} renamed /mcu/TXD0_{B1}
- net /PWR/CC1 renamed /usb/CC1
- net /PWR/CC2 renamed /usb/CC2
- net /PWR/D+_{J} renamed /usb/D+_{J}
- net /PWR/D-_{J} renamed /usb/D-_{J}
- net /PWR/EN_{3.3V} renamed /3v3/EN_{3.3V}
- net /PWR/FB_{3.3V} renamed /3v3/FB_{3.3V}
- net /PWR/GATE renamed /usb/GATE
- net /PWR/L1_{3.3V} renamed /3v3/L1_{3.3V}
- net /PWR/L2_{3.3V} renamed /3v3/L2_{3.3V}
- net /PWR/MODE_{5V} renamed /5v/MODE_{5V}
- net /PWR/SOURCE renamed /usb/SOURCE
- net /PWR/SW_{5V} renamed /5v/SW_{5V}
- net /PWR/VAUX_{3.3V} renamed /3v3/VAUX_{3.3V}
- net /PWR/VBUS_{C} renamed /usb/VBUS_{C}
- net /PWR/VIN_{3.3V} renamed /3v3/VIN_{3.3V}
- net /PWR/VSET_{5V} renamed /5v/VSET_{5V}
- D3 pad 1: /MCU/HB -> /mcu/HB
- J4 pad 1: unconnected-(J103-Pin_1-Pad1) -> M1_{B}
- J4 pad 11: unconnected-(J103-Pin_11-Pad11) -> GND
- J4 pad 12: unconnected-(J103-Pin_12-Pad12) -> +5V
- J4 pad 13: unconnected-(J103-Pin_13-Pad13) -> GND
- J4 pad 14: unconnected-(J103-Pin_14-Pad14) -> +5V
- J4 pad 15: unconnected-(J103-Pin_15-Pad15) -> GND
- J4 pad 16: unconnected-(J103-Pin_16-Pad16) -> +5V
- J4 pad 17: unconnected-(J103-Pin_17-Pad17) -> GND
- J4 pad 19: unconnected-(J103-Pin_19-Pad19) -> H1_{B}
- J4 pad 2: unconnected-(J103-Pin_2-Pad2) -> M1_{A}
- J4 pad 20: unconnected-(J103-Pin_20-Pad20) -> H1_{C}
- J4 pad 21: unconnected-(J103-Pin_21-Pad21) -> H1_{A}
- J4 pad 22: unconnected-(J103-Pin_22-Pad22) -> H1_{D}
- J4 pad 23: unconnected-(J103-Pin_23-Pad23) -> H10_{A}
- J4 pad 24: unconnected-(J103-Pin_24-Pad24) -> H10_{B}
- J4 pad 25: unconnected-(J103-Pin_25-Pad25) -> H10_{D}
- J4 pad 26: unconnected-(J103-Pin_26-Pad26) -> H10_{C}
- J4 pad 3: unconnected-(J103-Pin_3-Pad3) -> M1_{C}
- J4 pad 4: unconnected-(J103-Pin_4-Pad4) -> M1_{D}
- J4 pad 5: unconnected-(J103-Pin_5-Pad5) -> M10_{C}
- J4 pad 6: unconnected-(J103-Pin_6-Pad6) -> M10_{B}
- J4 pad 7: unconnected-(J103-Pin_7-Pad7) -> M10_{D}
- J4 pad 8: unconnected-(J103-Pin_8-Pad8) -> M10_{A}
- J4 pad 9: unconnected-(J103-Pin_9-Pad9) -> GND
- J5 pad 1: unconnected-(J102-Pin_1-Pad1) -> +3V3
- J5 pad 2: unconnected-(J102-Pin_2-Pad2) -> EN_{HV}
- J5 pad 3: unconnected-(J102-Pin_3-Pad3) -> V_{BUS}
- J5 pad 4: unconnected-(J102-Pin_4-Pad4) -> V_{BUS}
- J5 pad 5: unconnected-(J102-Pin_5-Pad5) -> PGOOD_{LM5155}
- J5 pad 6: unconnected-(J102-Pin_6-Pad6) -> GND
- U3 pad 10: M1_{B} -> M10_{D}
- U3 pad 11: M1_{D} -> M10_{A}
- U3 pad 12: M1_{A} -> EN_{HV}
- U3 pad 15: unconnected-(U153-GPIO3-Pad15) -> GPIO3
- U3 pad 17: EN_{HV} -> H1_{B}
- U3 pad 18: M10_{C} -> H1_{C}
- U3 pad 19: M10_{B} -> H1_{A}
- U3 pad 20: M10_{D} -> H1_{D}
- U3 pad 21: M10_{A} -> H10_{A}
- U3 pad 22: H1_{C} -> H10_{B}
- U3 pad 23: H1_{B} -> H10_{D}
- U3 pad 24: H1_{D} -> H10_{C}
- U3 pad 25: H1_{A} -> PGOOD_{LM5155}
- U3 pad 28: H10_{A} -> PD_{INT}
- U3 pad 29: H10_{D} -> USB_{~{OE}}
- U3 pad 30: H10_{B} -> PD_{FLT}
- U3 pad 31: H10_{C} -> /mcu/HB
- U3 pad 32: /MCU/MTCK -> MTCK
- U3 pad 33: /MCU/MTDO -> MTDO
- U3 pad 34: /MCU/MTDI -> MTDI
- U3 pad 35: /MCU/MTMS -> MTMS
- U3 pad 4: PD_{INT} -> M1_{B}
- U3 pad 5: PD_{FLT} -> M1_{A}
- U3 pad 6: USB_{~{OE}} -> M1_{C}
- U3 pad 7: /MCU/HB -> M1_{D}
- U3 pad 8: PGOOD_{LM5155} -> M10_{C}
- U3 pad 9: M1_{C} -> M10_{B}
Routing:
- net +3V3: track 118.0 -> 202.8 mm, vias 7 -> 11
- net EN_{MCU}: track 28.6 -> 101.9 mm, vias 2 -> 8
- net VCC_{UART}: track 0.00 -> 49.8 mm, vias 1 -> 3
- net PGOOD_{LM5155}: track 0.00 -> 43.1 mm, vias 0 -> 2
- net EN_{HV}: track 0.00 -> 41.2 mm, vias 0 -> 2
- net SDA: track 5.38 -> 46.3 mm
- net SCL: track 5.97 -> 46.0 mm
- net H1_{A}: track 0.00 -> 39.8 mm
- net H1_{D}: track 0.00 -> 38.5 mm
- net H1_{B}: track 0.00 -> 36.7 mm
- net /mcu/BOOT: track 4.53 -> 40.6 mm, vias 0 -> 2
- net H1_{C}: track 0.00 -> 35.8 mm
- net USB_{D-}: track 2.98 -> 38.2 mm, vias 0 -> 2
- net USB_{D+}: track 2.88 -> 36.8 mm, vias 0 -> 2
- net H10_{D}: track 15.6 -> 46.3 mm
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Other:
- board text added: "${TITLE}//REV ${REV}//${AUTHOR}"

Commit message: Rev B RC2
Parts:
- D104: value LED -> FAULT
Connections:
- J4 pad 17: GND -> unconnected-(J4-Pin_17-Pad17)
- J4 pad 9: GND -> unconnected-(J4-Pin_9-Pad9)
Changed lines of the file:
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@@
 	(net 94 "unconnected-(U3-GPIO45-Pad26)")
 	(net 95 "unconnected-(U3-GPIO46-Pad16)")
+	(net 96 "unconnected-(J4-Pin_17-Pad17)")
+	(net 97 "unconnected-(J4-Pin_9-Pad9)")
 	(footprint "TestPoint:TestPoint_Pad_D1.0mm"
 		(layer "F.Cu")
@@
 			)
 		)
-		(property "MFG Part No" ""
+		(property "MFG Part No" "TS3USB221AQRSERQ1"
 			(at 0 0 90)
 			(unlocked yes)
@@
 			)
 		)
-		(property "Value" "LED"
+		(property "Value" "FAULT"
 			(at 0 1.43 0)
-			(layer "F.Fab")
+			(layer "F.SilkS")
 			(effects
 				(font
@@
 			(layers "*.Cu" "*.Mask")
 			(remove_unused_layers no)
-			(net 45 "GND")
+			(net 97 "unconnected-(J4-Pin_9-Pad9)")
 			(pinfunction "Pin_9")
-			(pintype "passive")
+			(pintype "passive+no_connect")
 		)
 		(pad "10" thru_hole circle
@@
 			(net 90 "unconnected-(J4-Pin_10-Pad10)")
 			(pinfunction "Pin_10")
-			(pintype "passive")
+			(pintype "passive+no_connect")
 		)
 		(pad "11" thru_hole circle
@@
 			(layers "*.Cu" "*.Mask")
 			(remove_unused_layers no)
-			(net 45 "GND")
+			(net 96 "unconnected-(J4-Pin_17-Pad17)")
 			(pinfunction "Pin_17")
-			(pintype "passive")
+			(pintype "passive+no_connect")
 		)
 		(pad "18" thru_hole circle
@@
 			(net 89 "unconnected-(J4-Pin_18-Pad18)")
 			(pinfunction "Pin_18")
-			(pintype "passive")
+			(pintype "passive+no_connect")
 		)
 		(pad "19" thru_hole circle

Commit message: Rev B RC3
Parts:
- added R12: 10k, Resistor_SMD:R_0402_1005Metric, F.Cu at (122.6, 95.5)
- C124: footprint Capacitor_SMD:C_0603_1608Metric -> Capacitor_SMD:C_0402_1005Metric
- R127: value 100k -> 10k
- moved C124 0.20 mm to (135.3, 71.8)
Routing:
- net /mcu/BOOT: track 40.6 -> 44.5 mm
- net +3V3: track 202.8 -> 203.8 mm

Commit message: Final Rev B
Parts:
- moved C5 0.60 mm to (144.9, 113.0)
Routing:
- net +3V3: track 203.8 -> 204.4 mm
Changed lines of the file:
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@@
 		(sheetfile "mcu.kicad_sch")
 		(zone_connect 2)
-		(attr through_hole exclude_from_bom)
+		(attr through_hole exclude_from_pos_files exclude_from_bom)
 		(fp_line
 			(start -1.38 -1.38)
@@
 	(footprint "Capacitor_SMD:C_0402_1005Metric"
 		(layer "F.Cu")
-		(at 144.3 112.99)
+		(at 144.9 112.99)
 		(descr "Capacitor SMD 0402 (1005 Metric), square (rectangular) end terminal, IPC-7351 nominal, (Body size source: IPC-SM-782 page 76, https://www.pcb-3d.com/wordpress/wp-content/uploads/ipc-sm-782a_amendment_1_and_2.pdf), generated with kicad-footprint-generator")
 		(tags "capacitor")
@@
 		(sheetname "/mcu/")
 		(sheetfile "mcu.kicad_sch")
-		(attr smd)
+		(attr smd exclude_from_pos_files exclude_from_bom)
 		(fp_line
 			(start -2.075 -3.285)
@@
 		(sheetname "/mcu/")
 		(sheetfile "mcu.kicad_sch")
-		(attr through_hole)
+		(attr through_hole exclude_from_pos_files exclude_from_bom)
 		(fp_line
 			(start -1.38 -1.38)
@@
 		(sheetname "/mcu/")
 		(sheetfile "mcu.kicad_sch")
-		(attr through_hole)
+		(attr through_hole exclude_from_pos_files exclude_from_bom)
 		(fp_line
 			(start 5.83 35.69)
@@
 		(sheetname "/mcu/")
 		(sheetfile "mcu.kicad_sch")
-		(attr through_hole)
+		(attr through_hole exclude_from_pos_files exclude_from_bom)
 		(fp_line
 			(start 15.06 9.31)
@@
 	)
 	(segment
-		(start 143.82 112.99)
-		(end 141.75 112.99)
-		(width 0.5)
-		(layer "F.Cu")
-		(net 4)
-	)
-	(segment
-		(start 143.82 113.32)
-		(end 143.82 112.99)
-		(width 0.5)
-		(layer "F.Cu")
-		(net 4)
-	)
-	(segment
 		(start 138.425 76.1)
 		(end 137.874 76.651)
@@
 	)
 	(segment
-		(start 144.125 113.625)
-		(end 143.82 113.32)
-		(width 0.5)
-		(layer "F.Cu")
-		(net 4)
-	)
-	(segment
 		(start 117.607 99.507)
 		(end 117.875 99.775)
@@
 	)
 	(segment
+		(start 144.125 113.625)
+		(end 144.42 113.33)
+		(width 0.5)
+		(layer "F.Cu")
+		(net 4)
+	)
+	(segment
 		(start 120.89 112.99)
 		(end 121.29 112.99)
@@
 	)
 	(segment
+		(start 144.42 113.33)
+		(end 144.42 112.99)
+		(width 0.5)
+		(layer "F.Cu")
+		(net 4)
+	)
+	(segment
 		(start 153.9 82.05)
 		(end 153.9 97.14561)
@@
 	)
 	(segment
+		(start 141.75 112.99)
+		(end 144.42 112.99)
+		(width 0.5)
+		(layer "F.Cu")
+		(net 4)
+	)
+	(segment
 		(start 119.9 83.6)
 		(end 118.95 83.6)
@@
 	)
 	(via
-		(at 120.45 73.5)
+		(at 145.38 112.99)
 		(size 0.6)
 		(drill 0.3)
 		(layers "F.Cu" "B.Cu")
-		(free yes)
 		(net 45)
 	)
 	(via
-		(at 125 87.2)
+		(at 120.45 73.5)
 		(size 0.6)
 		(drill 0.3)
@@
 	)
 	(via
-		(at 155.2 112.6)
+		(at 125 87.2)
 		(size 0.6)
 		(drill 0.3)
@@
 	)
 	(via
-		(at 145.1 113)
+		(at 155.2 112.6)
 		(size 0.6)
 		(drill 0.3)

Commit message: HV converter Rev C redesign around LM5156
Parts:
- J101: footprint nixie_clock:USB_C_Receptacle_JAE_DX07S016JA1R1500 -> 0_nixie_clock:USB_C_Receptacle_JAE_DX07S016JA1R1500
- J2: footprint nixie_clock:Samtec_FTSH-105-01-L-DV-K_2x05_P1.27mm_Vertical_SMD -> 0_nixie_clock:Samtec_FTSH-105-01-L-DV-K_2x05_P1.27mm_Vertical_SMD
- L121, L131: footprint nixie_clock:L_Bourns_SRN5040TA -> 0_nixie_clock:L_Bourns_SRN5040TA
- SW1, SW2: footprint nixie_clock:SW_Panasonic_EVQ_4.9x4.9mm -> 0_nixie_clock:SW_Panasonic_EVQ_4.9x4.9mm
- U102: footprint nixie_clock:UQFN-10_1.5x2mm_P0.5mm_TI_RSE0010A -> 0_nixie_clock:UQFN-10_1.5x2mm_P0.5mm_TI_RSE0010A
- U103: footprint nixie_clock:QFN-24-1EP_4x4mm_P0.5mm_EP2.75x2.75mm_ThermalVias -> 0_nixie_clock:QFN-24-1EP_4x4mm_P0.5mm_EP2.75x2.75mm_ThermalVias
- U121: footprint nixie_clock:VQFN-15_2.5x3mm_TI_RNM0015A -> 0_nixie_clock:VQFN-15_2.5x3mm_TI_RNM0015A
- U3: footprint nixie_clock:ESP32-S3-WROOM-1 -> 0_nixie_clock:ESP32-S3-WROOM-1
Changed lines of the file:
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@@
 		)
 	)
-	(footprint "nixie_clock:USB_C_Receptacle_JAE_DX07S016JA1R1500"
+	(footprint "0_nixie_clock:USB_C_Receptacle_JAE_DX07S016JA1R1500"
 		(layer "F.Cu")
 		(at 103.55 79.4 -90)
@@
 		)
 	)
-	(footprint "nixie_clock:VQFN-15_2.5x3mm_TI_RNM0015A"
+	(footprint "0_nixie_clock:VQFN-15_2.5x3mm_TI_RNM0015A"
 		(layer "F.Cu")
 		(at 132.5 71.9 90)
@@
 		(embedded_fonts no)
 	)
-	(footprint "nixie_clock:UQFN-10_1.5x2mm_P0.5mm_TI_RSE0010A"
+	(footprint "0_nixie_clock:UQFN-10_1.5x2mm_P0.5mm_TI_RSE0010A"
 		(layer "F.Cu")
 		(at 120.8 83.6 90)
@@
 		)
 	)
-	(footprint "nixie_clock:QFN-24-1EP_4x4mm_P0.5mm_EP2.75x2.75mm_ThermalVias"
+	(footprint "0_nixie_clock:QFN-24-1EP_4x4mm_P0.5mm_EP2.75x2.75mm_ThermalVias"
 		(layer "F.Cu")
 		(at 116.55 74.5)
@@
 		(embedded_fonts no)
 	)
-	(footprint "nixie_clock:SW_Panasonic_EVQ_4.9x4.9mm"
+	(footprint "0_nixie_clock:SW_Panasonic_EVQ_4.9x4.9mm"
 		(layer "F.Cu")
 		(at 155.2 112.6 90)
@@
 		)
 	)
-	(footprint "nixie_clock:L_Bourns_SRN5040TA"
+	(footprint "0_nixie_clock:L_Bourns_SRN5040TA"
 		(layer "F.Cu")
 		(at 127.3 82.4 90)
@@
 		)
 	)
-	(footprint "nixie_clock:SW_Panasonic_EVQ_4.9x4.9mm"
+	(footprint "0_nixie_clock:SW_Panasonic_EVQ_4.9x4.9mm"
 		(layer "F.Cu")
 		(at 155.2 106.4 90)
@@
 		)
 	)
-	(footprint "nixie_clock:ESP32-S3-WROOM-1"
+	(footprint "0_nixie_clock:ESP32-S3-WROOM-1"
 		(layer "F.Cu")
 		(at 133 109 180)
@@
 		)
 	)
-	(footprint "nixie_clock:Samtec_FTSH-105-01-L-DV-K_2x05_P1.27mm_Vertical_SMD"
+	(footprint "0_nixie_clock:Samtec_FTSH-105-01-L-DV-K_2x05_P1.27mm_Vertical_SMD"
 		(layer "F.Cu")
 		(at 112.5 112)
@@
 		)
 	)
-	(footprint "nixie_clock:L_Bourns_SRN5040TA"
+	(footprint "0_nixie_clock:L_Bourns_SRN5040TA"
 		(layer "F.Cu")
 		(at 132.3 67.3)

Commit message: Main board Rev C
Parts:
- removed D121: 1N5819, Diode_SMD:D_SOD-123
- removed Q121: PMF170XP, Package_TO_SOT_SMD:SOT-323_SC-70
- added J131: I2C, Connector_PinHeader_2.54mm:PinHeader_1x04_P2.54mm_Vertical, F.Cu at (106.1, 87.2)
- added Q122: DMP3099L, Package_TO_SOT_SMD:SOT-23-3, F.Cu at (127.8, 65.8)
- added Q131: FDC6312P, Package_TO_SOT_SMD:SOT-23-6, F.Cu at (127.0, 69.7)
- added R129: 100k, Resistor_SMD:R_0402_1005Metric, F.Cu at (124.7, 67.6)
- added TP102: VBUS_{C}, TestPoint:TestPoint_Pad_D1.0mm, F.Cu at (109.2, 81.9)
- J3: footprint Connector_PinHeader_2.54mm:PinHeader_1x02_P2.54mm_Vertical -> Connector_PinHeader_1.27mm:PinHeader_1x02_P1.27mm_Vertical
- R101, R111: value 5.1k -> 20k; footprint Resistor_SMD:R_0603_1608Metric -> Resistor_SMD:R_0402_1005Metric
- R113: value 10k -> 100k
- R128: value 1k -> 2.4k
- R134: value 2.2k -> 5.6k
- moved R113 7.22 mm to (119.0, 66.4), turned to 90 degrees
- moved R8 6.51 mm to (114.7, 93.4)
- moved D3 6.23 mm to (116.0, 93.3)
- moved R123 4.00 mm to (124.7, 69.6), turned to 90 degrees
- moved R121 3.63 mm to (130.5, 71.1), turned to -90 degrees
- moved R122 3.57 mm to (129.4, 67.4), turned to 90 degrees
- moved C5 2.28 mm to (143.8, 111.0)
- moved C122 2.06 mm to (130.2, 73.6)
- moved C4 2.06 mm to (144.4, 112.2)
- moved D1 2.06 mm to (109.5, 101.7)
- moved D2 2.06 mm to (109.5, 100.0)
- moved R3 2.06 mm to (109.0, 103.0)
- moved R4 2.06 mm to (109.0, 98.7)
- moved C121 2.04 mm to (128.3, 73.8)
- moved C1 2.00 mm to (114.1, 104.7)
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Connections:
- net EN_{HV} renamed ~{EN}_{HV}
- net PGOOD_{LM5155} renamed PGOOD_{HV}
- net USB_{~{OE}} renamed ~{EN}_{USB}
- J4 pad 1: M1_{B} -> M1_{A}
- J4 pad 19: H1_{B} -> H10_{A}
- J4 pad 2: M1_{A} -> M10_{C}
- J4 pad 21: H1_{A} -> H10_{D}
- J4 pad 22: H1_{D} -> H1_{B}
- J4 pad 23: H10_{A} -> H10_{B}
- J4 pad 24: H10_{B} -> H1_{D}
- J4 pad 25: H10_{D} -> H10_{C}
- J4 pad 26: H10_{C} -> H1_{A}
- J4 pad 3: M1_{C} -> M1_{D}
- J4 pad 4: M1_{D} -> M10_{B}
- J4 pad 5: M10_{C} -> M1_{B}
- J4 pad 6: M10_{B} -> M10_{D}
- J4 pad 7: M10_{D} -> M1_{C}
- R122 pad 1: Net-(Q121-G) -> /3v3/G_{UART}
- U3 pad 10: M10_{D} -> M1_{C}
- U3 pad 17: H1_{B} -> H10_{A}
- U3 pad 19: H1_{A} -> H10_{D}
- U3 pad 20: H1_{D} -> H1_{B}
- U3 pad 21: H10_{A} -> H10_{B}
- U3 pad 22: H10_{B} -> H1_{D}
- U3 pad 23: H10_{D} -> H10_{C}
- U3 pad 24: H10_{C} -> H1_{A}
- U3 pad 4: M1_{B} -> M1_{A}
- U3 pad 5: M1_{A} -> M10_{C}
- U3 pad 6: M1_{C} -> M1_{D}
- U3 pad 7: M1_{D} -> M10_{B}
- U3 pad 8: M10_{C} -> M1_{B}
- U3 pad 9: M10_{B} -> M10_{D}
Routing:
- net H10_{D}: track 46.3 -> 37.3 mm
- net /mcu/HB: track 20.8 -> 12.7 mm
- net H10_{A}: track 42.7 -> 35.6 mm
- net /3v3/G_{UART}: track 0.00 -> 7.04 mm, vias 0 -> 2
- net SDA: track 46.3 -> 52.3 mm
- net SCL: track 46.0 -> 50.7 mm, vias 2 -> 3
- net Net-(Q121-G): track 4.10 -> 0.00 mm
- net M10_{C}: track 25.5 -> 21.6 mm
- net /3v3/G_{BUS}: track 0.00 -> 3.69 mm
- net +3V3: track 204.4 -> 208.1 mm
- net H1_{A}: track 39.8 -> 42.7 mm
- net V_{BUS}: track 101.9 -> 99.1 mm, vias 6 -> 4
- net M10_{D}: track 25.5 -> 22.7 mm
- net M1_{B}: track 27.8 -> 25.0 mm
- net VCC_{UART}: track 49.8 -> 47.1 mm
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Other:
- outline, holes or cut-outs redrawn
- board text added: "SCL"
- board text added: "SDA"
