File: pcb/main/main.kicad_pcb (KiCad board)
At the start: 2 copper layers, 70 x 65 mm, 103 parts, among them J1 UART, J101 USB_C_Receptacle_USB2.0_16P, J131 I2C, J2 JTAG, J3 JTAG SRC, J4 26 pin IDC, J5 Conn_01x06, Q101 Q_Dual_PMOS_S1G1S2G2D2D2D1D1, Q122 DMP3099L, Q131 FDC6312P, SW1 Boot, SW2 Reset, U1 74LVC1G17, U101 USBLC6-2SC6, U102 TS3USB221A, U103 CYPD3176, U121 TPS63070, U131 TPS629203, U2 74LVC1G17, U3 ESP32-S3-WROOM-1

Commit message: Updated schematic and improved make release to reduce manual jlc work
Parts:
- renumbered J131 to J6
Changed lines of the file:
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@@
 		(capping no)
 		(filling no)
-		(zone_defaults)
 		(pcbplotparams
 			(layerselection 0x00000000_00000000_55555555_5755f5ff)
@@
 			)
 		)
+		(property "shift_x" "0.95mm"
+			(at 0 0 270)
+			(unlocked yes)
+			(layer "F.Fab")
+			(hide yes)
+			(effects
+				(font
+					(size 1 1)
+					(thickness 0.15)
+				)
+			)
+		)
 		(property ki_fp_filters "USB*C*Receptacle*")
 		(sheetname "/usb/")
@@
 			)
 		)
+		(property "rotate" "270"
+			(at 0 0 90)
+			(unlocked yes)
+			(layer "F.Fab")
+			(hide yes)
+			(effects
+				(font
+					(size 1 1)
+					(thickness 0.15)
+				)
+			)
+		)
 		(sheetname "/usb/")
 		(sheetfile "usb.kicad_sch")
@@
 			)
 		)
+		(property "rotate" "270"
+			(at 0 0 90)
+			(unlocked yes)
+			(layer "F.Fab")
+			(hide yes)
+			(effects
+				(font
+					(size 1 1)
+					(thickness 0.15)
+				)
+			)
+		)
 		(property ki_fp_filters "*RNM0015A*")
 		(sheetname "/3v3/")
@@
 			)
 		)
+		(property "rotate" "180"
+			(at 0 0 0)
+			(unlocked yes)
+			(layer "F.Fab")
+			(hide yes)
+			(effects
+				(font
+					(size 1 1)
+					(thickness 0.15)
+				)
+			)
+		)
 		(sheetname "/3v3/")
 		(sheetfile "3v3.kicad_sch")
@@
 			)
 		)
+		(property "rotate" "270"
+			(at 0 0 0)
+			(unlocked yes)
+			(layer "F.Fab")
+			(hide yes)
+			(effects
+				(font
+					(size 1 1)
+					(thickness 0.15)
+				)
+			)
+		)
 		(sheetname "/usb/")
 		(sheetfile "usb.kicad_sch")
@@
 			)
 		)
+		(property "rotate" "270"
+			(at 0 0 180)
+			(unlocked yes)
+			(layer "F.Fab")
+			(hide yes)
+			(effects
+				(font
+					(size 1 1)
+					(thickness 0.15)
+				)
+			)
+		)
 		(property ki_fp_filters "SOT*583*")
 		(sheetname "/5v/")
@@
 			)
 		)
+		(property "rotate" "270"
+			(at 0 0 90)
+			(unlocked yes)
+			(layer "F.Fab")
+			(hide yes)
+			(effects
+				(font
+					(size 1 1)
+					(thickness 0.15)
+				)
+			)
+		)
 		(sheetname "/3v3/")
 		(sheetfile "3v3.kicad_sch")
@@
 			)
 		)
+		(property "shift_y" "-3.7mm"
+			(at 0 0 180)
+			(unlocked yes)
+			(layer "F.Fab")
+			(hide yes)
+			(effects
+				(font
+					(size 1 1)
+					(thickness 0.15)
+				)
+			)
+		)
 		(sheetname "/mcu/")
 		(sheetfile "mcu.kicad_sch")
@@
 		(descr "Through hole straight pin header, 1x04, 2.54mm pitch, single row")
 		(tags "Through hole pin header THT 1x04 2.54mm single row")
-		(property "Reference" "J131"
+		(property "Reference" "J6"
 			(at 0 -2.38 90)
 			(layer "F.SilkS")
@@
 			)
 		)
-		(attr through_hole)
+		(attr through_hole exclude_from_bom)
 		(duplicate_pad_numbers_are_jumpers no)
 		(fp_line
@@
 			)
 		)
+		(property "MFG Part No" "74LVC1G17"
+			(at 0 0 0)
+			(unlocked yes)
+			(layer "F.Fab")
+			(hide yes)
+			(effects
+				(font
+					(size 1 1)
+					(thickness 0.15)
+				)
+			)
+		)
+		(property "LCSC" ""
+			(at 0 0 0)
+			(unlocked yes)
+			(layer "F.Fab")
+			(hide yes)
+			(effects
+				(font
+					(size 1 1)
+					(thickness 0.15)
+				)
+			)
+		)
+		(property "rotate" "270"
+			(at 0 0 0)
+			(unlocked yes)
+			(layer "F.Fab")
+			(hide yes)
+			(effects
+				(font
+					(size 1 1)
+					(thickness 0.15)
+				)
+			)
+		)
 		(property ki_fp_filters "SOT?23* SOT?553* Texas?R-PDSO-G5?DCK* Texas?R-PDSO-N5?DRL* Texas?X2SON*0.8x0.8mm*P0.48mm*")
 		(sheetname "/mcu/")
@@
 			)
 		)
+		(property "rotate" "270"
+			(at 0 0 0)
+			(unlocked yes)
+			(layer "F.Fab")
+			(hide yes)
+			(effects
+				(font
+					(size 1 1)
+					(thickness 0.15)
+				)
+			)
+		)
 		(property ki_fp_filters "SOT?23*")
 		(sheetname "/usb/")
@@
 			)
 		)
-		(property "MFG Part No" ""
+		(property "MFG Part No" "74LVC1G17"
 			(at 0 0 180)
 			(unlocked yes)
@@
 			)
 		)
+		(property "rotate" "270"
+			(at 0 0 180)
+			(unlocked yes)
+			(layer "F.Fab")
+			(hide yes)
+			(effects
+				(font
+					(size 1 1)
+					(thickness 0.15)
+				)
+			)
+		)
 		(property ki_fp_filters "SOT?23* SOT?553* Texas?R-PDSO-G5?DCK* Texas?R-PDSO-N5?DRL* Texas?X2SON*0.8x0.8mm*P0.48mm*")
 		(sheetname "/mcu/")
@@
 			)
 		)
-		(property "MFG Part No" ""
+		(property "MFG Part No" "S6B-XH-A"
 			(at 0 0 180)
 			(unlocked yes)
@@
 	)
 	(segment
+		(start 124.728939 65.671061)
+		(end 125.55 64.85)
+		(width 0.5)
+		(layer "F.Cu")
+		(net "/3v3/G_{BUS}")
+	)
+	(segment
+		(start 125.55 64.85)
+		(end 126.6625 64.85)
+		(width 0.5)
+		(layer "F.Cu")
+		(net "/3v3/G_{BUS}")
+	)
+	(segment
+		(start 124.728939 67.09)
+		(end 124.728939 65.671061)
+		(width 0.5)
+		(layer "F.Cu")
+		(net "/3v3/G_{BUS}")
+	)
+	(segment
 		(start 127.899997 92.400003)
 		(end 127.9 92.4)
@@
 	)
 	(segment
+		(start 126.028939 70.8)
+		(end 126.028939 71.462499)
+		(width 0.5)
+		(layer "F.Cu")
+		(net "/3v3/G_{UART}")
+	)
+	(segment
+		(start 126.47894 71.9125)
+		(end 127.381623 71.9125)
+		(width 0.5)
+		(layer "F.Cu")
+		(net "/3v3/G_{UART}")
+	)
+	(segment
+		(start 126.028939 71.462499)
+		(end 126.47894 71.9125)
+		(width 0.5)
+		(layer "F.Cu")
+		(net "/3v3/G_{UART}")
+	)
+	(segment
+		(start 127.928939 71.365184)
+		(end 127.928939 70.8)
+		(width 0.5)
+		(layer "F.Cu")
+		(net "/3v3/G_{UART}")
+	)
+	(segment
+		(start 129.4 67.91)
+		(end 129.4 68.6)
+		(width 0.2)
+		(layer "F.Cu")
+		(net "/3v3/G_{UART}")
+	)
+	(segment
+		(start 127.381623 71.9125)
+		(end 127.928939 71.365184)
+		(width 0.5)
+		(layer "F.Cu")
+		(net "/3v3/G_{UART}")
+	)
+	(via
+		(at 129.4 68.6)
+		(size 0.6)
+		(drill 0.3)
+		(layers "F.Cu" "B.Cu")
+		(net "/3v3/G_{UART}")
+	)
+	(via
+		(at 127.928939 70.8)
+		(size 0.6)
+		(drill 0.3)
+		(layers "F.Cu" "B.Cu")
+		(net "/3v3/G_{UART}")
+	)
+	(segment
+		(start 127.928939 70.8)
+		(end 129.4 69.32894)
+		(width 0.2)
+		(layer "B.Cu")
+		(net "/3v3/G_{UART}")
+	)
+	(segment
+		(start 129.4 69.32894)
+		(end 129.4 68.6)
+		(width 0.2)
+		(layer "B.Cu")
+		(net "/3v3/G_{UART}")
+	)
+	(segment
+		(start 126.978939 70.8)
+		(end 126.978939 68.525)
+		(width 0.5)
+		(layer "F.Cu")
+		(net "/3v3/S_{UART}")
+	)
+	(segment
 		(start 157.634744 105.4)
 		(end 145.75 105.4)
@@
 		(net "Net-(D3-A)")
 	)
-	(segment
-		(start 126.978939 70.8)
-		(end 126.978939 68.525)
-		(width 0.5)
-		(layer "F.Cu")
-		(net "/3v3/S_{UART}")
-	)
-	(segment
-		(start 126.028939 70.8)
-		(end 126.028939 71.462499)
-		(width 0.5)
-		(layer "F.Cu")
-		(net "/3v3/G_{UART}")
-	)
-	(segment
-		(start 126.47894 71.9125)
-		(end 127.381623 71.9125)
-		(width 0.5)
-		(layer "F.Cu")
-		(net "/3v3/G_{UART}")
-	)
-	(segment
-		(start 126.028939 71.462499)
-		(end 126.47894 71.9125)
-		(width 0.5)
-		(layer "F.Cu")
-		(net "/3v3/G_{UART}")
-	)
-	(segment
-		(start 127.928939 71.365184)
-		(end 127.928939 70.8)
-		(width 0.5)
-		(layer "F.Cu")
-		(net "/3v3/G_{UART}")
-	)
-	(segment
-		(start 129.4 67.91)
-		(end 129.4 68.6)
-		(width 0.2)
-		(layer "F.Cu")
-		(net "/3v3/G_{UART}")
-	)
-	(segment
-		(start 127.381623 71.9125)
-		(end 127.928939 71.365184)
-		(width 0.5)
-		(layer "F.Cu")
-		(net "/3v3/G_{UART}")
-	)
-	(via
-		(at 129.4 68.6)
-		(size 0.6)
-		(drill 0.3)
-		(layers "F.Cu" "B.Cu")
-		(net "/3v3/G_{UART}")
-	)
-	(via
-		(at 127.928939 70.8)
-		(size 0.6)
-		(drill 0.3)
-		(layers "F.Cu" "B.Cu")
-		(net "/3v3/G_{UART}")
-	)
-	(segment
-		(start 127.928939 70.8)
-		(end 129.4 69.32894)
-		(width 0.2)
-		(layer "B.Cu")
-		(net "/3v3/G_{UART}")
-	)
-	(segment
-		(start 129.4 69.32894)
-		(end 129.4 68.6)
-		(width 0.2)
-		(layer "B.Cu")
-		(net "/3v3/G_{UART}")
-	)
-	(segment
-		(start 124.728939 65.671061)
-		(end 125.55 64.85)
-		(width 0.5)
-		(layer "F.Cu")
-		(net "/3v3/G_{BUS}")
-	)
-	(segment
-		(start 125.55 64.85)
-		(end 126.6625 64.85)
-		(width 0.5)
-		(layer "F.Cu")
-		(net "/3v3/G_{BUS}")
-	)
-	(segment
-		(start 124.728939 67.09)
-		(end 124.728939 65.671061)
-		(width 0.5)
-		(layer "F.Cu")
-		(net "/3v3/G_{BUS}")
-	)
 	(zone

Commit message: More schematic and parts tweaks
Parts:
- removed R133: 5.6k, Resistor_SMD:R_0402_1005Metric
- C101: footprint Capacitor_SMD:C_0805_2012Metric_Pad1.18x1.45mm_HandSolder -> Capacitor_SMD:C_0805_2012Metric
- C4: footprint Capacitor_SMD:C_0603_1608Metric -> Capacitor_SMD:C_1206_3216Metric
- R132: value 75k -> 80.6k
- moved TP1 2.98 mm to (150.5, 111.5)
- moved C4 1.84 mm to (146.0, 111.3), turned to -90 degrees
- moved C101 0.05 mm to (103.7, 67.1)
Connections:
- R132 pad 1: Net-(R132-Pad1) -> GND
Routing:
- net +3V3: track 208.1 -> 211.4 mm
- net Net-(R132-Pad1): track 0.89 -> 0.00 mm
- net GND: vias 54 -> 52
