File: pcb/main/3v3.kicad_sch (KiCad schematic)
At the start: 21 parts, among them Q121 PMF170XP, U121 TPS63070

Commit message: Rev B RC2
Parts:
- R127: value 100k -> 10k; LCSC C25741 -> C25744; MFG Part No 0402WGF1003TCE -> 0402WGF1002TCE
Changed lines of the file:
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@@
 			)
 		)
-		(property "Value" "100k"
+		(property "Value" "10k"
 			(at 183.134 91.44 0)
 			(effects
@@
 			)
 		)
-		(property "MFG Part No" "0402WGF1003TCE"
+		(property "MFG Part No" "0402WGF1002TCE"
 			(at 181.61 90.17 0)
 			(effects
@@
 			)
 		)
-		(property "LCSC" "C25741"
+		(property "LCSC" "C25744"
 			(at 181.61 90.17 0)
 			(effects

Commit message: Rev B RC3
Parts:
- C124: footprint Capacitor_SMD:C_0603_1608Metric -> Capacitor_SMD:C_0402_1005Metric; LCSC C59461 -> C15525; MFG Part No CL10A226MQ8NRNC -> CL05A106MQ5NUNC
Changed lines of the file:
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@@
 			)
 		)
-		(property "Footprint" "Capacitor_SMD:C_0603_1608Metric"
+		(property "Footprint" "Capacitor_SMD:C_0402_1005Metric"
 			(at 169.8752 88.9 0)
 			(effects
@@
 			)
 		)
-		(property "MFG Part No" "CL10A226MQ8NRNC"
+		(property "MFG Part No" "CL05A106MQ5NUNC"
 			(at 168.91 85.09 0)
 			(effects
@@
 			)
 		)
-		(property "LCSC" "C59461"
+		(property "LCSC" "C15525"
 			(at 168.91 85.09 0)
 			(effects

Commit message: HV converter Rev C redesign around LM5156
Parts:
- L121: footprint nixie_clock:L_Bourns_SRN5040TA -> 0_nixie_clock:L_Bourns_SRN5040TA
- U121: footprint nixie_clock:VQFN-15_2.5x3mm_TI_RNM0015A -> 0_nixie_clock:VQFN-15_2.5x3mm_TI_RNM0015A; symbol nixie_clock:TPS63070 -> 0_nixie_clock:TPS63070

Commit message: Main board Rev C
Parts:
- removed D121: 1N5819, Diode_SMD:D_SOD-123, symbol Device:D_Schottky
- removed Q121: PMF170XP, Package_TO_SOT_SMD:SOT-323_SC-70, symbol Transistor_FET:Q_PMOS_GSD
- added Q122: DMP3099L, Package_TO_SOT_SMD:SOT-23-3, symbol Transistor_FET:Q_PMOS_GSD
- added Q131: FDC6312P, Package_TO_SOT_SMD:SOT-23-6, symbol Transistor_FET:Q_Dual_PMOS_G1S2G2D2S1D1
- added R129: 100k, Resistor_SMD:R_0402_1005Metric, symbol Device:R
- R126: LCSC C25794 -> C25783; MFG Part No 0402WGF5102TCE -> 0402WGF3902TCE
- R128: value 1k -> 2.4k; LCSC C11702 -> C25882; MFG Part No 0402WGF1001TCE -> 0402WGF2401TCE
Connections:
- net VCC_{UART}: now also Q131.6 (D), R129.2
- net VIN_{3.3V}: now also Q122.2 (S), Q131.4 (D)
- net V_{BUS}: now also Q122.3 (D)
- net G_{UART}: now reaches R122.1
- net G_{UART}: now also Q131.1 (G), Q131.3 (G)
- new net G_{BUS}: Q122.1 (G), R129.1
- new net S_{UART}: Q131.2 (S), Q131.5 (S)
Other:
- moved on the sheet: R122, R123

Commit message: Updated schematic and improved make release to reduce manual jlc work
Parts:
- Q122: rotate (none) -> 180
- Q131, U121: rotate (none) -> 270
Changed lines of the file:
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@@
+			)
+		)
+		(property "rotate" "270"
+			(at 144.78 90.17 0)
+			(hide yes)
+			(show_name no)
+			(do_not_autoplace no)
+			(effects
+				(font
+					(size 1.27 1.27)
+				)
 			)
 		)
@@
 		)
 		(property "LCSC" "C241767"
+			(at 92.71 60.96 0)
+			(hide yes)
+			(show_name no)
+			(do_not_autoplace no)
+			(effects
+				(font
+					(size 1.27 1.27)
+				)
+			)
+		)
+		(property "rotate" "270"
 			(at 92.71 60.96 0)
 			(hide yes)
@@
 			)
 		)
+		(property "rotate" "180"
+			(at 92.71 96.52 0)
+			(hide yes)
+			(show_name no)
+			(do_not_autoplace no)
+			(effects
+				(font
+					(size 1.27 1.27)
+				)
+			)
+		)
 		(pin "1"
 		)
@@
 			(at 92.71 73.66 0)
 			(hide yes)
+			(show_name no)
+			(do_not_autoplace no)
+			(effects
+				(font
+					(size 1.27 1.27)
+				)
+			)
+		)
+		(property "rotate" "270"
+			(at 92.71 73.66 0)
+			(hide yes)

Commit message: More schematic and parts tweaks
Parts:
- R123: LCSC C25741 -> C93945; MFG Part No 0402WGF1003TCE -> RC0402FR-07120KL
Changed lines of the file:
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@@
 			)
 		)
-		(property "MFG Part No" "0402WGF1003TCE"
+		(property "MFG Part No" "RC0402FR-07120KL"
 			(at 111.76 63.5 0)
 			(hide yes)
@@
 			)
 		)
-		(property "LCSC" "C25741"
+		(property "LCSC" "C93945"
 			(at 111.76 63.5 0)
 			(hide yes)

Commit message: Parts updates, a few board tweaks
Parts:
- C123: MFG Part No CL05B104KO5NNNC -> CL05B104KB54PNC
Connections:
- net FB_{3.3V} renamed FB_{3V3}
- net L1_{3.3V} renamed SW_{3V3A}
- net L2_{3.3V} renamed SW_{3V3B}
- net VAUX_{3.3V} renamed V_{AUX}
- net VCC_{UART} renamed V_{UART}
- net VIN_{3.3V} renamed V_{IN3.3V}
Changed lines of the file:
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@@
 		)
 	)
-	(label "FB_{3.3V}"
+	(label "FB_{3V3}"
 		(at 162.56 90.17 0)
 		(effects
@@
 		)
 	)
-	(label "VIN_{3.3V}"
+	(label "V_{IN3.3V}"
 		(at 105.41 82.55 0)
 		(effects
@@
 		)
 	)
-	(label "L1_{3.3V}"
+	(label "SW_{3V3A}"
 		(at 130.81 73.66 0)
 		(effects
@@
 		)
 	)
-	(label "VAUX_{3.3V}"
+	(label "V_{AUX}"
 		(at 127 105.41 0)
 		(effects
@@
 		)
 	)
-	(label "L2_{3.3V}"
+	(label "SW_{3V3B}"
 		(at 153.67 73.66 0)
 		(effects
@@
 		(in_pos_files yes)
 		(dnp no)
-		(fields_autoplaced yes)
 		(property "Reference" "#PWR0212"
 			(at 95.25 59.69 0)
@@
 			)
 		)
-		(property "Value" "VCC_{UART}"
-			(at 95.25 50.8 0)
+		(property "Value" "V_{UART}"
+			(at 97.028 53.34 0)
 			(show_name no)
 			(do_not_autoplace no)
@@
 					(size 1.27 1.27)
 				)
+				(justify left)
 			)
 		)
@@
 			)
 		)
-		(property "MFG Part No" "CL05B104KO5NNNC"
+		(property "MFG Part No" "CL05B104KB54PNC"
 			(at 132.08 109.22 0)
 			(hide yes)
@@
 		(in_pos_files yes)
 		(dnp no)
-		(fields_autoplaced yes)
 		(property "Reference" "#PWR0208"
 			(at 77.47 95.25 0)
@@
 			)
 		)
-		(property "Value" "VCC_{UART}"
-			(at 77.47 104.14 0)
+		(property "Value" "V_{UART}"
+			(at 78.232 102.616 0)
 			(show_name no)
 			(do_not_autoplace no)
@@
 					(size 1.27 1.27)
 				)
+				(justify right)
 			)
 		)
