File: pcb/main/3v3.kicad_sch (KiCad schematic)
At the start: 22 parts, among them Q122 DMP3099L, Q131 FDC6312P, U121 TPS63070

Commit message: Update release process, update analysis to use INS-1 throughout
Parts:
- R123: LCSC C93945 -> C60491; MFG Part No RC0402FR-07120KL -> RC0402FR-07100KL
Changed lines of the file:
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@@
 			)
 		)
-		(property "MFG Part No" "RC0402FR-07120KL"
+		(property "MFG Part No" "RC0402FR-07100KL"
 			(at 111.76 63.5 0)
 			(hide yes)
@@
 			)
 		)
-		(property "LCSC" "C93945"
+		(property "LCSC" "C60491"
 			(at 111.76 63.5 0)
 			(hide yes)

Commit message: Update IN-12 model to the one we've created
Parts:
- R122, R129: MFG Part No 0402WGF1003TCE -> RC0402FR-07100KL
Changed lines of the file:
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@@
 			)
 		)
-		(property "MFG Part No" "0402WGF1003TCE"
+		(property "MFG Part No" "RC0402FR-07100KL"
 			(at 83.82 96.52 0)
 			(hide yes)
@@
 			)
 		)
-		(property "MFG Part No" "0402WGF1003TCE"
+		(property "MFG Part No" "RC0402FR-07100KL"
 			(at 83.82 67.31 0)
 			(hide yes)
