File: pcb/main/5v.kicad_sch (KiCad schematic)
At the start: 12 parts, among them U131 TPS629203

Commit message: HV converter Rev C redesign around LM5156
Parts:
- L131: footprint nixie_clock:L_Bourns_SRN5040TA -> 0_nixie_clock:L_Bourns_SRN5040TA
- U131: symbol nixie_clock:TPS629203 -> 0_nixie_clock:TPS629203

Commit message: Main board Rev C
Parts:
- R134: value 2.2k -> 5.6k; LCSC C25879 -> C25908; MFG Part No 0402WGF2201TCE -> 0402WGF5601TCE
Other:
- moved on the sheet: C131, C132, C133, D131, L131, R131, R132, R133, R134, TP131, TP132, U131

Commit message: Updated schematic and improved make release to reduce manual jlc work
Parts:
- U131: rotate (none) -> 270
Changed lines of the file:
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@@
+			)
+		)
+		(property "rotate" "270"
+			(at 68.58 48.26 0)
+			(hide yes)
+			(show_name no)
+			(do_not_autoplace no)
+			(effects
+				(font
+					(size 1.27 1.27)
+				)
 			)
 		)

Commit message: More schematic and parts tweaks
Parts:
- removed R133: 5.6k, Resistor_SMD:R_0402_1005Metric, symbol Device:R
- R132: value 75k -> 80.6k; LCSC C25798 -> C155698; MFG Part No 0402WGF7502TCE -> RC0402FR-0780K6L
Connections:
- net GND: now also R132.1
Changed lines of the file:
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@@
 	(symbol
 		(lib_id "power:GND")
-		(at 91.44 66.04 0)
+		(at 91.44 58.42 0)
 		(unit 1)
 		(body_style 1)
@@
 		(fields_autoplaced yes)
 		(property "Reference" "#PWR0248"
-			(at 91.44 72.39 0)
+			(at 91.44 64.77 0)
 			(hide yes)
 			(show_name no)
@@
 		)
 		(property "Value" "GND"
-			(at 91.44 71.12 0)
+			(at 91.44 63.5 0)
 			(hide yes)
 			(show_name no)
@@
 		)
 		(property "Footprint" ""
-			(at 91.44 66.04 0)
+			(at 91.44 58.42 0)
 			(hide yes)
 			(show_name no)
@@
 		)
 		(property "Datasheet" ""
-			(at 91.44 66.04 0)
+			(at 91.44 58.42 0)
 			(hide yes)
 			(show_name no)
@@
 		)
 		(property "Description" "Power symbol creates a global label with name \"GND\" , ground"
-			(at 91.44 66.04 0)
+			(at 91.44 58.42 0)
 			(hide yes)
 			(show_name no)
@@
 		)
 		(property "MFG Part No" ""
-			(at 91.44 66.04 0)
+			(at 91.44 58.42 0)
 			(hide yes)
 			(show_name no)
@@
 		)
 		(property "LCSC" ""
-			(at 91.44 66.04 0)
+			(at 91.44 58.42 0)
 			(hide yes)
 			(show_name no)
@@
 			)
 		)
-		(property "Value" "75k"
+		(property "Value" "80.6k"
 			(at 92.964 55.88 0)
 			(show_name no)
@@
 			)
 		)
-		(property "MFG Part No" "0402WGF7502TCE"
+		(property "MFG Part No" "RC0402FR-0780K6L"
 			(at 91.44 54.61 0)
 			(hide yes)
@@
 			)
 		)
-		(property "LCSC" "C25798"
+		(property "LCSC" "C155698"
 			(at 91.44 54.61 0)
 			(hide yes)
@@
 					(unit 1)
 				)
-			)
-		)
-	)
-	(symbol
-		(lib_id "Device:R")
-		(at 91.44 62.23 180)
-		(unit 1)
-		(body_style 1)
-		(exclude_from_sim no)
-		(in_bom yes)
-		(on_board yes)
-		(in_pos_files yes)
-		(dnp no)
-		(property "Reference" "R133"
-			(at 92.964 60.96 0)
-			(show_name no)
-			(do_not_autoplace no)
-			(effects
-				(font
-					(size 1.27 1.27)
-				)
-				(justify right)
-			)
-		)
-		(property "Value" "5.6k"
-			(at 92.964 63.5 0)
-			(show_name no)
-			(do_not_autoplace no)
-			(effects
-				(font
-					(size 1.27 1.27)
-				)
-				(justify right)
-			)
-		)
-		(property "Footprint" "Resistor_SMD:R_0402_1005Metric"
-			(at 93.218 62.23 90)
-			(hide yes)
-			(show_name no)
-			(do_not_autoplace no)
-			(effects
-				(font
-					(size 1.27 1.27)
-				)
-			)
-		)
-		(property "Datasheet" ""
-			(at 91.44 62.23 0)
-			(hide yes)
-			(show_name no)
-			(do_not_autoplace no)
-			(effects
-				(font
-					(size 1.27 1.27)
-				)
-			)
-		)
-		(property "Description" "Resistor"
-			(at 91.44 62.23 0)
-			(hide yes)
-			(show_name no)
-			(do_not_autoplace no)
-			(effects
-				(font
-					(size 1.27 1.27)
-				)
-			)
-		)
-		(property "MFG Part No" "0402WGF5601TCE"
-			(at 91.44 62.23 0)
-			(hide yes)
-			(show_name no)
-			(do_not_autoplace no)
-			(effects
-				(font
-					(size 1.27 1.27)
-				)
-			)
-		)
-		(property "LCSC" "C25908"
-			(at 91.44 62.23 0)
-			(hide yes)
-			(show_name no)
-			(do_not_autoplace no)
-			(effects
-				(font
-					(size 1.27 1.27)
-				)
-			)
-		)
-		(pin "1"
-		)
-		(pin "2"
-		)
-		(instances
-			(project "main"
-				(path "/f225fc02-d36f-4469-bac4-82a576baae3a/6897350a-6b24-4568-8df0-70384d2ca7c6"
-					(reference "R133")
-					(unit 1)
-				)

Commit message: Parts updates, a few board tweaks
Connections:
- net MODE_{5V} renamed FB_{MODE}
- net VSET_{5V} renamed FB_{5V}
Changed lines of the file:
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@@
 		)
 	)
-	(label "MODE_{5V}"
+	(label "FB_{MODE}"
 		(at 44.45 50.8 0)
 		(effects
@@
 		)
 	)
-	(label "VSET_{5V}"
+	(label "FB_{5V}"
 		(at 86.36 50.8 0)
 		(effects
