File: pcb/main/usb.kicad_sch (KiCad schematic)
At the start: 32 parts, among them J101 USB_C_Receptacle_USB2.0_16P, Q101 Q_Dual_PMOS_S1G1S2G2D2D2D1D1, U101 USBLC6-2SC6, U102 TS3USB221A, U103 CYPD3176

Commit message: Rev B RC1
Changed lines of the file:
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@@
 	)
 	(junction
+		(at 82.55 118.11)
+		(diameter 0)
+		(color 0 0 0 0)
+	)
+	(junction
 		(at 99.06 35.56)
 		(diameter 0)
@@
 	(wire
 		(pts
+			(xy 86.36 118.11) (xy 82.55 118.11)
+		)
+		(stroke
+			(width 0)
+			(type default)
+		)
+	)
+	(wire
+		(pts
 			(xy 102.87 97.79) (xy 99.06 97.79)
 		)
@@
 	)
 	(global_label "PD_{INT}"
-		(shape input)
+		(shape output)
 		(at 189.23 87.63 0)
 		(fields_autoplaced yes)
@@
 					(unit 1)
 				)
+			)
+		)
+	)
+	(symbol
+		(lib_id "power:PWR_FLAG")
+		(at 86.36 118.11 180)
+		(unit 1)
+		(exclude_from_sim no)
+		(in_bom yes)
+		(on_board yes)
+		(dnp no)
+		(fields_autoplaced yes)
+		(property "Reference" "#FLG01"
+			(at 86.36 120.015 0)
+			(effects
+				(font
+					(size 1.27 1.27)
+				)
+				(hide yes)
+			)
+		)
+		(property "Value" "PWR_FLAG"
+			(at 86.36 123.19 0)
+			(effects
+				(font
+					(size 1.27 1.27)
+				)
+				(hide yes)
+			)
+		)
+		(property "Footprint" ""
+			(at 86.36 118.11 0)
+			(effects
+				(font
+					(size 1.27 1.27)
+				)
+				(hide yes)
+			)
+		)
+		(property "Datasheet" "~"
+			(at 86.36 118.11 0)
+			(effects
+				(font
+					(size 1.27 1.27)
+				)
+				(hide yes)
+			)
+		)
+		(property "Description" "Special symbol for telling ERC where power comes from"
+			(at 86.36 118.11 0)
+			(effects
+				(font
+					(size 1.27 1.27)
+				)
+				(hide yes)
+			)
+		)
+		(property "MFG Part No" ""
+			(at 86.36 118.11 0)
+			(effects
+				(font
+					(size 1.27 1.27)
+				)
+				(hide yes)
+			)
+		)
+		(property "LCSC" ""
+			(at 86.36 118.11 0)
+			(effects
+				(font
+					(size 1.27 1.27)
+				)
+				(hide yes)
+			)
+		)
+		(pin "1"
+		)
+		(instances
+			(project "main"
+				(path "/f225fc02-d36f-4469-bac4-82a576baae3a/f8973f07-5632-4b97-a3ce-a5e33fa36ed2"
+					(reference "#FLG01")
+					(unit 1)
+				)

Commit message: Rev B RC2
Parts:
- D104: value LED -> FAULT
- U102: MFG Part No (none) -> TS3USB221AQRSERQ1
Changed lines of the file:
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@@
 			)
 		)
-		(property "Value" "LED"
+		(property "Value" "FAULT"
 			(at 194.31 105.7274 90)
 			(effects
@@
 			)
 		)
-		(property "MFG Part No" ""
+		(property "MFG Part No" "TS3USB221AQRSERQ1"
 			(at 115.57 133.35 0)
 			(effects

Commit message: Fix part # typos
Parts:
- R107, R109: LCSC C25905 -> C25882; MFG Part No 0402WGF5101TCE -> 0402WGF2401TCE
Changed lines of the file:
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@@
 			)
 		)
-		(property "MFG Part No" "0402WGF5101TCE"
+		(property "MFG Part No" "0402WGF2401TCE"
 			(at 177.8 128.27 0)
 			(effects
@@
 			)
 		)
-		(property "LCSC" "C25905"
+		(property "LCSC" "C25882"
 			(at 177.8 128.27 0)
 			(effects
@@
 			)
 		)
-		(property "MFG Part No" "0402WGF5101TCE"
+		(property "MFG Part No" "0402WGF2401TCE"
 			(at 167.64 135.89 0)
 			(effects
@@
 			)
 		)
-		(property "LCSC" "C25905"
+		(property "LCSC" "C25882"
 			(at 167.64 135.89 0)
 			(effects

Commit message: HV converter Rev C redesign around LM5156
Parts:
- J101: footprint nixie_clock:USB_C_Receptacle_JAE_DX07S016JA1R1500 -> 0_nixie_clock:USB_C_Receptacle_JAE_DX07S016JA1R1500
- U102: footprint nixie_clock:UQFN-10_1.5x2mm_P0.5mm_TI_RSE0010A -> 0_nixie_clock:UQFN-10_1.5x2mm_P0.5mm_TI_RSE0010A; symbol nixie_clock:TS3USB221A -> 0_nixie_clock:TS3USB221A
- U103: footprint nixie_clock:QFN-24-1EP_4x4mm_P0.5mm_EP2.75x2.75mm_ThermalVias -> 0_nixie_clock:QFN-24-1EP_4x4mm_P0.5mm_EP2.75x2.75mm_ThermalVias; symbol nixie_clock:CYPD3176 -> 0_nixie_clock:CYPD3176
Connections:
- net USB_{~{OE}} renamed ~{EN}_{USB}

Commit message: Main board Rev C
Parts:
- added TP102: VBUS_{C}, TestPoint:TestPoint_Pad_D1.0mm, symbol Connector:TestPoint
- C104, C107: Note (none) -> Chosen with the expectation of above nominal derating in th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
- Q101: MFG Part No DMP3085LSD-13 -> FDS4935A
- R101, R111: value 5.1k -> 20k; footprint Resistor_SMD:R_0603_1608Metric -> Resistor_SMD:R_0402_1005Metric; LCSC C23186 -> C25765; MFG Part No 0603WAF5101T5E -> 0402WGF2002TCE
- R113: value 10k -> 100k; LCSC C25744 -> C25741; MFG Part No 0402WGF1002TCE -> 0402WGF1003TCE
Connections:
- net GND: now also J101.SH (SHIELD); no longer J101.S1 (SHIELD)
- net VBUS_{C}: now also TP102.1
Changed lines of the file:
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@@
 			)
 		)
-		(property "Value" "5.1k"
+		(property "Value" "20k"
 			(at 89.154 40.64 0)
 			(show_name no)
@@
 			)
 		)
-		(property "Footprint" "Resistor_SMD:R_0603_1608Metric"
+		(property "Footprint" "Resistor_SMD:R_0402_1005Metric"
 			(at 89.408 39.37 90)
 			(hide yes)
@@
 			)
 		)
-		(property "MFG Part No" "0603WAF5101T5E"
+		(property "MFG Part No" "0402WGF2002TCE"
 			(at 87.63 39.37 0)
 			(hide yes)
@@
 			)
 		)
-		(property "LCSC" "C23186"
+		(property "LCSC" "C25765"
 			(at 87.63 39.37 0)
 			(hide yes)
@@
 		(dnp no)
 		(property "Reference" "U103"
-			(at 149.352 74.422 0)
+			(at 149.352 72.644 0)
 			(show_name no)
 			(do_not_autoplace no)
@@
 		)
 		(property "Value" "CYPD3176"
-			(at 151.638 76.708 0)
+			(at 151.638 74.93 0)
 			(show_name no)
 			(do_not_autoplace no)
@@
 			)
 		)
-		(property "Datasheet" "${KIPRJMOD}/../docs/datasheets/infineon-cypd3176-24lqxq-datasheet-en.pdf"
+		(property "Datasheet" "${KIPRJMOD}/../../docs/datasheets/infineon-cypd3176-24lqxq-datasheet-en.pdf"
 			(at 165.1 115.57 0)
 			(hide yes)
@@
 			)
 		)
-		(property "MFG Part No" "DMP3085LSD-13"
+		(property "MFG Part No" "FDS4935A"
 			(at 177.8 39.37 0)
 			(hide yes)
@@
 			)
 		)
+		(property "Note" "Chosen with the expectation of above nominal derating in this application. Expect ~200nF actual capacitance"
+			(at 138.43 39.37 0)
+			(hide yes)
+			(show_name no)
+			(do_not_autoplace no)
+			(effects
+				(font
+					(size 1.27 1.27)
+				)
+			)
+		)
 		(pin "1"
 		)
@@
 			)
 		)
-		(property "Value" "10k"
+		(property "Value" "100k"
 			(at 211.074 41.91 0)
 			(show_name no)
@@
 			)
 		)
-		(property "MFG Part No" "0402WGF1002TCE"
+		(property "MFG Part No" "0402WGF1003TCE"
 			(at 209.55 40.64 0)
 			(hide yes)
@@
 			)
 		)
-		(property "LCSC" "C25744"
+		(property "LCSC" "C25741"
 			(at 209.55 40.64 0)
 			(hide yes)
@@
 	)
 	(symbol
+		(lib_id "Connector:TestPoint")
+		(at 105.41 35.56 0)
+		(unit 1)
+		(body_style 1)
+		(exclude_from_sim no)
+		(in_bom no)
+		(on_board yes)
+		(in_pos_files yes)
+		(dnp no)
+		(property "Reference" "TP102"
+			(at 102.362 30.226 0)
+			(show_name no)
+			(do_not_autoplace no)
+			(effects
+				(font
+					(size 1.27 1.27)
+				)
+				(justify left)
+			)
+		)
+		(property "Value" "VBUS_{C}"
+			(at 106.6799 30.48 90)
+			(hide yes)
+			(show_name no)
+			(do_not_autoplace no)
+			(effects
+				(font
+					(size 1.27 1.27)
+				)
+				(justify left)
+			)
+		)
+		(property "Footprint" "TestPoint:TestPoint_Pad_D1.0mm"
+			(at 110.49 35.56 0)
+			(hide yes)
+			(show_name no)
+			(do_not_autoplace no)
+			(effects
+				(font
+					(size 1.27 1.27)
+				)
+			)
+		)
+		(property "Datasheet" ""
+			(at 110.49 35.56 0)
+			(hide yes)
+			(show_name no)
+			(do_not_autoplace no)
+			(effects
+				(font
+					(size 1.27 1.27)
+				)
+			)
+		)
+		(property "Description" "test point"
+			(at 105.41 35.56 0)
+			(hide yes)
+			(show_name no)
+			(do_not_autoplace no)
+			(effects
+				(font
+					(size 1.27 1.27)
+				)
+			)
+		)
+		(property "MFG Part No" ""
+			(at 105.41 35.56 0)
+			(hide yes)
+			(show_name no)
+			(do_not_autoplace no)
+			(effects
+				(font
+					(size 1.27 1.27)
+				)
+			)
+		)
+		(property "LCSC" ""
+			(at 105.41 35.56 0)
+			(hide yes)
+			(show_name no)
+			(do_not_autoplace no)
+			(effects
+				(font
+					(size 1.27 1.27)
+				)
+			)
+		)
+		(pin "1"
+		)
+		(instances
+			(project "main"
+				(path "/f225fc02-d36f-4469-bac4-82a576baae3a/f8973f07-5632-4b97-a3ce-a5e33fa36ed2"
+					(reference "TP102")
+					(unit 1)
+				)
+			)
+		)
+	)
+	(symbol
 		(lib_id "Device:D_Zener")
 		(at 102.87 71.12 270)
@@
 			)
 		)
-		(property "MFG Part No" "DMP3085LSD-13"
+		(property "MFG Part No" "FDS4935A"
 			(at 154.94 39.37 0)
 			(hide yes)
@@
 			)
 		)
+		(property "Note" "Chosen with the expectation of above nominal derating in this application. Expect ~200nF actual capacitance"
+			(at 185.42 40.64 0)
+			(hide yes)
+			(show_name no)
+			(do_not_autoplace no)
+			(effects
+				(font
+					(size 1.27 1.27)
+				)
+			)
+		)
 		(pin "1"
 		)
@@
 			)
 		)
-		(property "Datasheet" "ts3usb221a.pdf"
+		(property "Datasheet" "${KIPRJMOD}/../../docs/datasheets/ts3usb221a.pdf"
 			(at 115.824 133.096 0)
 			(hide yes)
@@
 			)
 		)
-		(property "Value" "5.1k"
+		(property "Value" "20k"
 			(at 198.374 41.91 0)
 			(show_name no)
@@
 			)
 		)
-		(property "Footprint" "Resistor_SMD:R_0603_1608Metric"
+		(property "Footprint" "Resistor_SMD:R_0402_1005Metric"
 			(at 198.628 40.64 90)
 			(hide yes)
@@
 			)
 		)
-		(property "MFG Part No" "0603WAF5101T5E"
+		(property "MFG Part No" "0402WGF2002TCE"
 			(at 196.85 40.64 0)
 			(hide yes)
@@
 			)
 		)
-		(property "LCSC" "C23186"
+		(property "LCSC" "C25765"
 			(at 196.85 40.64 0)
 			(hide yes)
@@
 		(pin "B1"
 		)
-		(pin "S1"
+		(pin "SH"
 		)
 		(pin "B6"

Commit message: Updated schematic and improved make release to reduce manual jlc work
Parts:
- J101: shift_x (none) -> 0.95mm
- Q101, U101, U103: rotate (none) -> 270
Changed lines of the file:
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@@
 			)
 		)
+		(property "rotate" "270"
+			(at 165.1 90.17 0)
+			(hide yes)
+			(show_name no)
+			(do_not_autoplace no)
+			(effects
+				(font
+					(size 1.27 1.27)
+				)
+			)
+		)
 		(pin "8"
 		)
@@
 			)
 		)
+		(property "rotate" "270"
+			(at 177.8 39.37 90)
+			(hide yes)
+			(show_name no)
+			(do_not_autoplace no)
+			(effects
+				(font
+					(size 1.27 1.27)
+				)
+			)
+		)
 		(pin "8"
 		)
@@
 			)
 		)
+		(property "rotate" "270"
+			(at 154.94 39.37 90)
+			(hide yes)
+			(show_name no)
+			(do_not_autoplace no)
+			(effects
+				(font
+					(size 1.27 1.27)
+				)
+			)
+		)
 		(pin "8"
 		)
@@
 			)
 		)
+		(property "rotate" "270"
+			(at 107.95 95.25 0)
+			(hide yes)
+			(show_name no)
+			(do_not_autoplace no)
+			(effects
+				(font
+					(size 1.27 1.27)
+				)
+			)
+		)
 		(pin "3"
 		)
@@
 			(at 82.55 95.25 0)
 			(hide yes)
+			(show_name no)
+			(do_not_autoplace no)
+			(effects
+				(font
+					(size 1.27 1.27)
+				)
+			)
+		)
+		(property "shift_x" "0.95mm"
+			(at 82.55 95.25 0)
+			(hide yes)

Commit message: More schematic and parts tweaks
Parts:
- J101: LCSC (none) -> C3197885
- U102: LCSC (none) -> C128396; MFG Part No TS3USB221AQRSERQ1 -> TS3USB221ARSER; rotate (none) -> 270
Changed lines of the file:
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@@
 			)
 		)
-		(property "MFG Part No" "TS3USB221AQRSERQ1"
+		(property "MFG Part No" "TS3USB221ARSER"
 			(at 115.57 133.35 0)
 			(hide yes)
@@
 			)
 		)
-		(property "LCSC" ""
+		(property "LCSC" "C128396"
+			(at 115.57 133.35 0)
+			(hide yes)
+			(show_name no)
+			(do_not_autoplace no)
+			(effects
+				(font
+					(size 1.27 1.27)
+				)
+			)
+		)
+		(property "rotate" "270"
 			(at 115.57 133.35 0)
 			(hide yes)
@@
 			)
 		)
-		(property "LCSC" ""
+		(property "LCSC" "C3197885"
 			(at 82.55 95.25 0)
 			(hide yes)

Commit message: Parts updates, a few board tweaks
Parts:
- C101: footprint Capacitor_SMD:C_0805_2012Metric_Pad1.18x1.45mm_HandSolder -> Capacitor_SMD:C_0805_2012Metric
- C106, C108: LCSC C1525 -> C307331; MFG Part No CL05B104KO5NNNC -> CL05B104KB54PNC
- R104: value 49.9K -> 100k; LCSC C25897 -> C25741; MFG Part No 0402WGF4992TCE -> 0402WGF1003TCE
Connections:
- net FB_{ISINKF}: now reaches R106.2, R107.1, U103.16 (ISNK_FINE)
- net FB_{VBUSMAX}: now reaches R108.2, R109.1, U103.2 (VBUS_MAX)
- net V_{CCD}: now reaches C103.1, U103.24 (VCCD)
- net GATE renamed G_{USB}
- net SOURCE renamed S_{USB}
- net VBUS_{C} renamed V_{BUSC}
- net VDDD renamed V_{DDD}
