File: pcb/main/usb.kicad_sch (KiCad schematic)
At the start: 33 parts, among them J101 USB_C_Receptacle_USB2.0_16P, Q101 Q_Dual_PMOS_S1G1S2G2D2D2D1D1, U101 USBLC6-2SC6, U102 TS3USB221A, U103 CYPD3176

Commit message: Add digikey profile, fix incorrect mpn on main
Parts:
- R105: MFG Part No 0402WGF1002TCE -> 0402WGF1001TCE
Changed lines of the file:
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@@
 			)
 		)
-		(property "MFG Part No" "0402WGF1002TCE"
+		(property "MFG Part No" "0402WGF1001TCE"
 			(at 160.02 48.26 0)
 			(hide yes)

Commit message: Update IN-12 model to the one we've created
Parts:
- D104: MFG Part No 2 (none) -> LTST-C190KRKT
- Q101: value Q_Dual_PMOS_S1G1S2G2D2D2D1D1 -> FDS4935A
- R101, R111: MFG Part No 0402WGF2002TCE -> RC0402FR-0720KL
- R102, R103: MFG Part No 0402WGF1002TCE -> RC0402JR-0710KL
- R104, R113: MFG Part No 0402WGF1003TCE -> RC0402FR-07100KL
- R106, R108: MFG Part No 0402WGF5101TCE -> RC0402FR-075K1L
Changed lines of the file:
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@@
 			)
 		)
-		(property "MFG Part No" "0402WGF1002TCE"
+		(property "MFG Part No" "RC0402JR-0710KL"
 			(at 128.27 39.37 0)
 			(hide yes)
@@
 			)
 		)
-		(property "MFG Part No" "0402WGF2002TCE"
+		(property "MFG Part No" "RC0402FR-0720KL"
 			(at 87.63 39.37 0)
 			(hide yes)
@@
 			)
 		)
-		(property "MFG Part No" "0402WGF5101TCE"
+		(property "MFG Part No" "RC0402FR-075K1L"
 			(at 167.64 128.27 0)
 			(hide yes)
@@
 			)
 		)
+		(property "MFG Part No 2" "LTST-C190KRKT"
+			(at 190.5 102.87 90)
+			(hide yes)
+			(show_name no)
+			(do_not_autoplace no)
+			(effects
+				(font
+					(size 1.27 1.27)
+				)
+			)
+		)
 		(pin "1"
 		)
@@
 			)
 		)
-		(property "Value" "Q_Dual_PMOS_S1G1S2G2D2D2D1D1"
+		(property "Value" "FDS4935A"
 			(at 177.8 31.75 90)
 			(hide yes)
@@
 			)
 		)
-		(property "MFG Part No" "0402WGF1002TCE"
+		(property "MFG Part No" "RC0402JR-0710KL"
 			(at 87.63 132.08 0)
 			(hide yes)
@@
 			)
 		)
-		(property "MFG Part No" "0402WGF5101TCE"
+		(property "MFG Part No" "RC0402FR-075K1L"
 			(at 177.8 120.65 0)
 			(hide yes)
@@
 			)
 		)
-		(property "MFG Part No" "0402WGF1003TCE"
+		(property "MFG Part No" "RC0402FR-07100KL"
 			(at 209.55 40.64 0)
 			(hide yes)
@@
 			)
 		)
-		(property "Value" "Q_Dual_PMOS_S1G1S2G2D2D2D1D1"
+		(property "Value" "FDS4935A"
 			(at 154.94 31.75 90)
 			(hide yes)
@@
 			)
 		)
-		(property "MFG Part No" "0402WGF2002TCE"
+		(property "MFG Part No" "RC0402FR-0720KL"
 			(at 196.85 40.64 0)
 			(hide yes)
@@
 			)
 		)
-		(property "MFG Part No" "0402WGF1003TCE"
+		(property "MFG Part No" "RC0402FR-07100KL"
 			(at 160.02 40.64 0)
 			(hide yes)

Commit message: Bump main to Rev D1, add EN_USB jumper to board, fix UART LED locations.
Parts:
- added J7: EN_{USB}, Connector_PinHeader_1.27mm:PinHeader_1x02_P1.27mm_Vertical, symbol Connector_Generic:Conn_01x02
Connections:
- net GND: now also J7.1 (Pin_1)
- net ~{EN}_{USB}: now also J7.2 (Pin_2)
Changed lines of the file:
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@@
 	(wire
 		(pts
+			(xy 87.63 135.89) (xy 87.63 140.97)
+		)
+		(stroke
+			(width 0)
+			(type default)
+		)
+	)
+	(wire
+		(pts
 			(xy 128.27 44.45) (xy 138.43 44.45)
 		)
@@
 	)
 	(symbol
+		(lib_id "Connector_Generic:Conn_01x02")
+		(at 82.55 143.51 180)
+		(unit 1)
+		(body_style 1)
+		(exclude_from_sim no)
+		(in_bom yes)
+		(on_board yes)
+		(in_pos_files yes)
+		(dnp no)
+		(property "Reference" "J7"
+			(at 79.248 140.716 0)
+			(show_name no)
+			(do_not_autoplace no)
+			(effects
+				(font
+					(size 1.27 1.27)
+				)
+			)
+		)
+		(property "Value" "EN_{USB}"
+			(at 77.978 143.002 0)
+			(show_name no)
+			(do_not_autoplace no)
+			(effects
+				(font
+					(size 1.27 1.27)
+				)
+			)
+		)
+		(property "Footprint" "Connector_PinHeader_1.27mm:PinHeader_1x02_P1.27mm_Vertical"
+			(at 82.55 143.51 0)
+			(hide yes)
+			(show_name no)
+			(do_not_autoplace no)
+			(effects
+				(font
+					(size 1.27 1.27)
+				)
+			)
+		)
+		(property "Datasheet" ""
+			(at 82.55 143.51 0)
+			(hide yes)
+			(show_name no)
+			(do_not_autoplace no)
+			(effects
+				(font
+					(size 1.27 1.27)
+				)
+			)
+		)
+		(property "Description" "Generic connector, single row, 01x02, script generated (kicad-library-utils/schlib/autogen/connector/)"
+			(at 82.55 143.51 0)
+			(hide yes)
+			(show_name no)
+			(do_not_autoplace no)
+			(effects
+				(font
+					(size 1.27 1.27)
+				)
+			)
+		)
+		(property "MFG Part No" "M50-3530242"
+			(at 82.55 143.51 0)
+			(hide yes)
+			(show_name no)
+			(do_not_autoplace no)
+			(effects
+				(font
+					(size 1.27 1.27)
+				)
+			)
+		)
+		(property "LCSC" ""
+			(at 82.55 143.51 0)
+			(hide yes)
+			(show_name no)
+			(do_not_autoplace no)
+			(effects
+				(font
+					(size 1.27 1.27)
+				)
+			)
+		)
+		(property "Note" "Close with M50-1900005 or equivelent"
+			(at 82.55 143.51 0)
+			(hide yes)
+			(show_name no)
+			(do_not_autoplace no)
+			(effects
+				(font
+					(size 1.27 1.27)
+				)
+			)
+		)
+		(pin "1"
+		)
+		(pin "2"
+		)
+		(instances
+			(project "main"
+				(path "/f225fc02-d36f-4469-bac4-82a576baae3a/f8973f07-5632-4b97-a3ce-a5e33fa36ed2"
+					(reference "J7")
+					(unit 1)
+				)
+			)
+		)
+	)
+	(symbol
 		(lib_id "power:GND")
 		(at 87.63 50.8 0)
@@
 					(unit 1)
 				)
+			)
+		)
+	)
+	(symbol
+		(lib_id "power:GND")
+		(at 87.63 143.51 0)
+		(unit 1)
+		(body_style 1)
+		(exclude_from_sim no)
+		(in_bom yes)
+		(on_board yes)
+		(in_pos_files yes)
+		(dnp no)
+		(fields_autoplaced yes)
+		(property "Reference" "#PWR0114"
+			(at 87.63 149.86 0)
+			(hide yes)
+			(show_name no)
+			(do_not_autoplace no)
+			(effects
+				(font
+					(size 1.27 1.27)
+				)
+			)
+		)
+		(property "Value" "GND"
+			(at 87.63 148.59 0)
+			(hide yes)
+			(show_name no)
+			(do_not_autoplace no)
+			(effects
+				(font
+					(size 1.27 1.27)
+				)
+			)
+		)
+		(property "Footprint" ""
+			(at 87.63 143.51 0)
+			(hide yes)
+			(show_name no)
+			(do_not_autoplace no)
+			(effects
+				(font
+					(size 1.27 1.27)
+				)
+			)
+		)
+		(property "Datasheet" ""
+			(at 87.63 143.51 0)
+			(hide yes)
+			(show_name no)
+			(do_not_autoplace no)
+			(effects
+				(font
+					(size 1.27 1.27)
+				)
+			)
+		)
+		(property "Description" "Power symbol creates a global label with name \"GND\" , ground"
+			(at 87.63 143.51 0)
+			(hide yes)
+			(show_name no)
+			(do_not_autoplace no)
+			(effects
+				(font
+					(size 1.27 1.27)
+				)
+			)
+		)
+		(property "MFG Part No" ""
+			(at 87.63 143.51 0)
+			(hide yes)
+			(show_name no)
+			(do_not_autoplace no)
+			(effects
+				(font
+					(size 1.27 1.27)
+				)
+			)
+		)
+		(property "LCSC" ""
+			(at 87.63 143.51 0)
+			(hide yes)
+			(show_name no)
+			(do_not_autoplace no)
+			(effects
+				(font
+					(size 1.27 1.27)
+				)
+			)
+		)
+		(pin "1"
+		)
+		(instances
+			(project "main"
+				(path "/f225fc02-d36f-4469-bac4-82a576baae3a/f8973f07-5632-4b97-a3ce-a5e33fa36ed2"
+					(reference "#PWR0114")
+					(unit 1)
+				)

Commit message: Tweaks to the new jumper
Parts:
- J7: value EN_{USB} -> FLASH
Changed lines of the file:
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@@
 			)
 		)
-		(property "Value" "EN_{USB}"
+		(property "Value" "FLASH"
 			(at 77.978 143.002 0)
 			(show_name no)
