File: pcb/main/mcu.kicad_sch (KiCad schematic)
At the start: 32 parts, among them J1 UART, J2 JTAG, J3 JTAG SRC, J4 26 pin IDC, J5 Conn_01x06, J6 I2C, SW1 Boot, SW2 Reset, U1 74LVC1G17, U2 74LVC1G17, U3 ESP32-S3-WROOM-1

Commit message: More schematic and parts tweaks
Parts:
- C4: footprint Capacitor_SMD:C_0603_1608Metric -> Capacitor_SMD:C_1206_3216Metric; LCSC C59461 -> C5672; MFG Part No CL10A226MQ8NRNC -> CL31A226KPHNNNE
Changed lines of the file:
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@@
 			)
 		)
-		(property "Footprint" "Capacitor_SMD:C_0603_1608Metric"
+		(property "Footprint" "Capacitor_SMD:C_1206_3216Metric"
 			(at 129.2352 38.1 0)
 			(hide yes)
@@
 			)
 		)
-		(property "MFG Part No" "CL10A226MQ8NRNC"
+		(property "MFG Part No" "CL31A226KPHNNNE"
 			(at 128.27 34.29 0)
 			(hide yes)
@@
 			)
 		)
-		(property "LCSC" "C59461"
+		(property "LCSC" "C5672"
 			(at 128.27 34.29 0)
 			(hide yes)

Commit message: Parts updates, a few board tweaks
Parts:
- C1, C2, C3, C5: LCSC C1525 -> C307331; MFG Part No CL05B104KO5NNNC -> CL05B104KB54PNC
Connections:
- net VCC_{UART} renamed V_{UART}
Changed lines of the file:
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@@
 			)
 		)
-		(property "MFG Part No" "CL05B104KO5NNNC"
+		(property "MFG Part No" "CL05B104KB54PNC"
 			(at 139.7 34.29 0)
 			(hide yes)
@@
 			)
 		)
-		(property "LCSC" "C1525"
+		(property "LCSC" "C307331"
 			(at 139.7 34.29 0)
 			(hide yes)
@@
 		(in_pos_files yes)
 		(dnp no)
-		(fields_autoplaced yes)
 		(property "Reference" "#PWR0512"
 			(at 31.75 72.39 0)
@@
 			)
 		)
-		(property "Value" "VCC_{UART}"
-			(at 31.75 81.28 0)
+		(property "Value" "V_{UART}"
+			(at 32.512 79.756 0)
 			(show_name no)
 			(do_not_autoplace no)
@@
 					(size 1.27 1.27)
 				)
+				(justify right)
 			)
 		)
@@
 			)
 		)
-		(property "MFG Part No" "CL05B104KO5NNNC"
+		(property "MFG Part No" "CL05B104KB54PNC"
 			(at 69.85 68.58 0)
 			(hide yes)
@@
 			)
 		)
-		(property "LCSC" "C1525"
+		(property "LCSC" "C307331"
 			(at 69.85 68.58 0)
 			(hide yes)
@@
 			)
 		)
-		(property "MFG Part No" "CL05B104KO5NNNC"
+		(property "MFG Part No" "CL05B104KB54PNC"
 			(at 111.76 39.37 0)
 			(hide yes)
@@
 			)
 		)
-		(property "LCSC" "C1525"
+		(property "LCSC" "C307331"
 			(at 111.76 39.37 0)
 			(hide yes)
@@
 			)
 		)
-		(property "MFG Part No" "CL05B104KO5NNNC"
+		(property "MFG Part No" "CL05B104KB54PNC"
 			(at 44.45 31.75 0)
 			(hide yes)
@@
 			)
 		)
-		(property "LCSC" "C1525"
+		(property "LCSC" "C307331"
 			(at 44.45 31.75 0)
 			(hide yes)

Commit message: Improve several 3D models, design testing base plate
Parts:
- J2, J3, J4, J5, J6: now in the parts list
Changed lines of the file:
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@@
 		(body_style 1)
 		(exclude_from_sim no)
-		(in_bom no)
+		(in_bom yes)
 		(on_board yes)
 		(in_pos_files yes)
@@
 		(body_style 1)
 		(exclude_from_sim no)
-		(in_bom no)
+		(in_bom yes)
 		(on_board yes)
 		(in_pos_files yes)
@@
 		(body_style 1)
 		(exclude_from_sim no)
-		(in_bom no)
+		(in_bom yes)
 		(on_board yes)
 		(in_pos_files yes)
@@
 		(body_style 1)
 		(exclude_from_sim no)
-		(in_bom no)
+		(in_bom yes)
 		(on_board yes)
 		(in_pos_files yes)
@@
 		(body_style 1)
 		(exclude_from_sim no)
-		(in_bom no)
+		(in_bom yes)
 		(on_board yes)
 		(in_pos_files yes)

Commit message: Update ins1 tube model, update hv/main connector to 1 vbus, 2 gnd connections, update hv inhibit circuit to be default inhibit and require positive enable from MCU
Parts:
- J4: MFG Part No (none) -> 75869-105LF; Note (none) -> Mates with 71600-026LF
Connections:
- net GND: now also J4.10 (Pin_10), J4.17 (Pin_17), J4.18 (Pin_18), J4.9 (Pin_9), J5.4 (Pin_4)
- net V_{BUS}: no longer J5.4 (Pin_4)
- net ~{EN}_{HV} renamed EN_{HV}
- no-connect marks 8 -> 4

Commit message: Update IN-12 model to the one we've created
Parts:
- D1: MFG Part No 2 (none) -> LTST-C190KSKT
- R1: MFG Part No 0402WGF1500TCE -> RC0402JR-0710KL
- R10, R11, R12, R2, R9: MFG Part No 0402WGF1002TCE -> RC0402JR-0710KL
- R6: MFG Part No 0402WGF1003TCE -> RC0402FR-07100KL
- U1, U2: MFG Part No 74LVC1G17 -> 74LVC1G17GV,125
Changed lines of the file:
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@@
 			)
 		)
-		(property "MFG Part No" "0402WGF1002TCE"
+		(property "MFG Part No" "RC0402JR-0710KL"
 			(at 46.99 81.28 0)
 			(hide yes)
@@
 			)
 		)
+		(property "MFG Part No 2" " LTST-C190KSKT"
+			(at 66.04 36.83 90)
+			(hide yes)
+			(show_name no)
+			(do_not_autoplace no)
+			(effects
+				(font
+					(size 1.27 1.27)
+				)
+			)
+		)
 		(pin "2"
 		)
@@
 			)
 		)
-		(property "MFG Part No" "0402WGF1002TCE"
+		(property "MFG Part No" "RC0402JR-0710KL"
 			(at 190.5 90.17 0)
 			(hide yes)
@@
 			)
 		)
-		(property "MFG Part No" "0402WGF1002TCE"
+		(property "MFG Part No" "RC0402JR-0710KL"
 			(at 92.71 38.1 0)
 			(hide yes)
@@
 			)
 		)
-		(property "MFG Part No" "74LVC1G17"
+		(property "MFG Part No" "74LVC1G17GV,125"
 			(at 50.8 46.99 0)
 			(hide yes)
@@
 			)
 		)
-		(property "MFG Part No" "0402WGF1003TCE"
+		(property "MFG Part No" "RC0402FR-07100KL"
 			(at 63.5 116.84 0)
 			(hide yes)
@@
 			)
 		)
-		(property "MFG Part No" "74LVC1G17"
+		(property "MFG Part No" "74LVC1G17GV,125"
 			(at 60.96 77.47 0)
 			(hide yes)
@@
 			)
 		)
-		(property "MFG Part No" "0402WGF1002TCE"
+		(property "MFG Part No" "RC0402JR-0710KL"
 			(at 182.88 41.91 0)
 			(hide yes)
@@
 			)
 		)
-		(property "MFG Part No" "0402WGF1500TCE"
+		(property "MFG Part No" "RC0402JR-0710KL"
 			(at 40.64 58.42 0)
 			(hide yes)
@@
 			)
 		)
-		(property "MFG Part No" "0402WGF1002TCE"
+		(property "MFG Part No" "RC0402JR-0710KL"
 			(at 196.85 44.45 0)
 			(hide yes)
