File: docs/design_analysis/schematics/3v3.kicad_sch (KiCad schematic)
At the start: 16 parts, among them U302 TPS63070

Commit message: Main board Rev C
Parts:
- removed D_{3V3BUS}: 1N5819, Diode_SMD:D_SOD-123, symbol Device:D_Schottky
- added Q_{3V3BUS}: DMP3099L, Package_TO_SOT_SMD:SOT-323_SC-70, symbol Transistor_FET:Q_PMOS_GSD
- added R_{3V3BLEED}, R_{3V3BUS}: 100k, Resistor_SMD:R_0402_1005Metric, symbol Device:R
Connections:
- net GND: now also R_{3V3BLEED}.1
- net VCC_{UART}: now also R_{3V3BLEED}.2, R_{3V3BUS}.1
- net V_{BUS}: now also Q_{3V3BUS}.3 (D)
- net at C_{3V3I1}.1, C_{3V3I2}.1, Q_{3V3HDR}.2 (S)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: now also Q_{3V3BUS}.2 (S)
- new net: Q_{3V3BUS}.1 (G), R_{3V3BUS}.2
