File: pcb/face/face.kicad_pcb (KiCad board)
At the start: 2 copper layers, 140 x 70 mm, 26 parts, among them J1 26 pin IDC, J2 Phoenix MSTB, U1 K155ID1, U2 K155ID1, U3 K155ID1, U4 K155ID1

Commit message: Main board Rev C
Parts:
- C3: value 47uF -> 10uF; footprint 0_nixie_clock:CP_Radial_D6.3mm_P2.50mm -> Capacitor_THT:CP_Radial_D5.0mm_P2.00mm
- NX5, NX6: value IN-6 -> INS-1; footprint 0_nixie_clock:IN-6 -> 0_nixie_clock:INS-1_Recessed
- moved C3 0.50 mm to (145.0, 66.0)
Routing:
- net +5V: track 189.7 -> 192.4 mm, vias 3 -> 1
- net /NX6_{A}: track 9.45 -> 8.59 mm
- net /NX5_{A}: track 9.45 -> 8.59 mm
