File: pcb/face/face.kicad_pcb (KiCad board)
At the start: 2 copper layers, 140 x 70 mm, 26 parts, among them J1 26 pin IDC, J2 Phoenix MSTB, U1 K155ID1, U2 K155ID1, U3 K155ID1, U4 K155ID1

Commit message: Update fab attributes, update silscreen to include step
Other:
- board text added: "${TITLE}//REV ${REV}${STEP}//${AUTHOR}"
- board text removed: "${TITLE}//REV ${REV}//${AUTHOR}"
Changed lines of the file:
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@@
 		(sheetname "/")
 		(sheetfile "face.kicad_sch")
+		(attr through_hole)
 		(duplicate_pad_numbers_are_jumpers no)
 		(fp_rect
@@
 		(sheetname "/")
 		(sheetfile "face.kicad_sch")
+		(attr through_hole)
 		(duplicate_pad_numbers_are_jumpers no)
 		(fp_rect
@@
 		(layer "Edge.Cuts")
 	)
-	(gr_text "${TITLE}//REV ${REV}//${AUTHOR}\n"
+	(gr_text "${TITLE}//REV ${REV}${STEP}//${AUTHOR}\n"
 		(at 151 74 0)
 		(layer "B.SilkS")

Commit message: Update ins1 tube model, update hv/main connector to 1 vbus, 2 gnd connections, update hv inhibit circuit to be default inhibit and require positive enable from MCU
Parts:
- R1, R2, R3, R4: value 8.2k -> 7.5k
- R5, R6: value 120k -> 240k
Connections:
- J1 pad 10: unconnected-(J1-Pin_10-Pad10) -> GND
- J1 pad 17: unconnected-(J1-Pin_17-Pad17) -> GND
- J1 pad 18: unconnected-(J1-Pin_18-Pad18) -> GND
- J1 pad 9: unconnected-(J1-Pin_9-Pad9) -> GND
