File: pcb/face/face.kicad_sch (KiCad schematic)
At the start: 25 parts, among them J104 Conn_02x13_Counter_Clockwise, U1 K155ID1, U2 K155ID1, U3 K155ID1, U4 K155ID1

Commit message: Split project into 3
Other:
- removed sheet HV
- removed sheet MCU
- removed sheet PWR
- title: ${TITLE} -> (none)
- moved on the sheet: C1, C2, C3, C4, H2, H3, H4, H5, J104, NX1, NX2, NX3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

Commit message: Rev B RC1
Parts:
- added J2: Phoenix MSTB, Connector_Phoenix_MSTB:PhoenixContact_MSTBVA_2,5_3-G-5,08_1x03_P5.08mm_Vertical, symbol Connector_Generic:Conn_01x03
- J1: renamed from J104; value Conn_02x13_Counter_Clockwise -> 26 pin IDC
- renumbered C2 to C1, C1 to C2, C4 to C3, C3 to C4, H2 to H1, H4 to H2, H5 to H4, NX5 to NX1, NX1 to NX3, NX6 to NX4, NX4 to NX5, NX3 to NX6, R5 to R1, R1 to R3, R6 to R4, R4 to R5, R3 to R6, U2 to U1, U1 to U2, U4 to U3, U3 to U4
Connections:
- net +170V: now also J2.1 (Pin_1)
- net GND: now also J2.3 (Pin_3)
- no-connect marks 6 -> 11

Commit message: Final Rev B
Parts:
- J1, J2, NX1, NX2, NX3, NX4, NX5, NX6, U1, U2, U3, U4: now left out of the parts list
Changed lines of the file:
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@@
 		(unit 1)
 		(exclude_from_sim no)
-		(in_bom yes)
+		(in_bom no)
 		(on_board yes)
 		(dnp no)
@@
 		(unit 1)
 		(exclude_from_sim no)
-		(in_bom yes)
+		(in_bom no)
 		(on_board yes)
 		(dnp no)
@@
 			)
 		)
+		(property "LCSC" ""
+			(at 46.99 91.44 0)
+			(effects
+				(font
+					(size 1.27 1.27)
+				)
+				(hide yes)
+			)
+		)
 		(pin "3"
 		)
@@
 		(unit 1)
 		(exclude_from_sim no)
-		(in_bom yes)
+		(in_bom no)
 		(on_board yes)
 		(dnp no)
@@
 		(unit 1)
 		(exclude_from_sim no)
-		(in_bom yes)
+		(in_bom no)
 		(on_board yes)
 		(dnp no)
@@
 		(unit 1)
 		(exclude_from_sim no)
-		(in_bom yes)
+		(in_bom no)
 		(on_board yes)
 		(dnp no)
@@
 		(unit 1)
 		(exclude_from_sim no)
-		(in_bom yes)
+		(in_bom no)
 		(on_board yes)
 		(dnp no)
@@
 		(unit 1)
 		(exclude_from_sim no)
-		(in_bom yes)
+		(in_bom no)
 		(on_board yes)
 		(dnp no)
@@
 		(unit 1)
 		(exclude_from_sim no)
-		(in_bom yes)
+		(in_bom no)
 		(on_board yes)
 		(dnp no)
@@
 		(unit 1)
 		(exclude_from_sim no)
-		(in_bom yes)
+		(in_bom no)
 		(on_board yes)
 		(dnp no)
@@
 		(unit 1)
 		(exclude_from_sim no)
-		(in_bom yes)
+		(in_bom no)
 		(on_board yes)
 		(dnp no)
@@
 			)
 		)
+		(property "LCSC" ""
+			(at 129.54 90.17 0)
+			(effects
+				(font
+					(size 1.27 1.27)
+				)
+				(hide yes)
+			)
+		)
 		(pin "3"
 		)
@@
 		(unit 1)
 		(exclude_from_sim no)
-		(in_bom yes)
+		(in_bom no)
 		(on_board yes)
 		(dnp no)
@@
 			)
 		)
+		(property "LCSC" ""
+			(at 129.54 40.64 0)
+			(effects
+				(font
+					(size 1.27 1.27)
+				)
+				(hide yes)
+			)
+		)
 		(pin "3"
 		)
@@
 		(unit 1)
 		(exclude_from_sim no)
-		(in_bom yes)
+		(in_bom no)
 		(on_board yes)
 		(dnp no)

Commit message: HV converter Rev C redesign around LM5156
Parts:
- C1, C2, C3, C4: footprint nixie_clock:C_Rect_L5.1mm_W3.2mm_P2.54mm_Goldmax -> 0_nixie_clock:C_Rect_L5.1mm_W3.2mm_P2.54mm_Goldmax
- NX1, NX4: footprint nixie_clock:IN-6 -> 0_nixie_clock:IN-6; symbol nixie_clock:IN-6 -> 0_nixie_clock:IN-6
- NX2, NX3, NX5, NX6: footprint nixie_clock:IN-12-DSUB -> 0_nixie_clock:IN-12-DSUB; symbol nixie_clock:IN-12B -> 0_nixie_clock:IN-12B
- U1, U2, U3, U4: footprint nixie_clock:DIP16 -> 0_nixie_clock:DIP16; symbol nixie_clock:K155ID1 -> 0_nixie_clock:K155ID1
Changed lines of the file:
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@@
 			)
 		)
-		(property "Footprint" "nixie_clock:C_Rect_L5.1mm_W3.2mm_P2.54mm_Goldmax"
+		(property "Footprint" "0_nixie_clock:C_Rect_L5.1mm_W3.2mm_P2.54mm_Goldmax"
 			(at 107.6452 85.09 0)
 			(effects
@@
 	)
 	(symbol
-		(lib_id "nixie_clock:K155ID1")
+		(lib_id "0_nixie_clock:K155ID1")
 		(at 46.99 41.91 0)
 		(unit 1)
@@
 			)
 		)
-		(property "Footprint" "nixie_clock:DIP16"
+		(property "Footprint" "0_nixie_clock:DIP16"
 			(at 47.752 38.1 0)
 			(effects
@@
 	)
 	(symbol
-		(lib_id "nixie_clock:K155ID1")
+		(lib_id "0_nixie_clock:K155ID1")
 		(at 46.99 91.44 0)
 		(unit 1)
@@
 			)
 		)
-		(property "Footprint" "nixie_clock:DIP16"
+		(property "Footprint" "0_nixie_clock:DIP16"
 			(at 47.752 87.63 0)
 			(effects
@@
 			)
 		)
-		(property "Footprint" "nixie_clock:C_Rect_L5.1mm_W3.2mm_P2.54mm_Goldmax"
+		(property "Footprint" "0_nixie_clock:C_Rect_L5.1mm_W3.2mm_P2.54mm_Goldmax"
 			(at 107.6452 35.56 0)
 			(effects
@@
 	)
 	(symbol
-		(lib_id "nixie_clock:IN-6")
+		(lib_id "0_nixie_clock:IN-6")
 		(at 204.47 59.69 0)
 		(unit 1)
@@
 			)
 		)
-		(property "Footprint" "nixie_clock:IN-6"
+		(property "Footprint" "0_nixie_clock:IN-6"
 			(at 205.232 55.88 0)
 			(effects
@@
 	)
 	(symbol
-		(lib_id "nixie_clock:IN-12B")
+		(lib_id "0_nixie_clock:IN-12B")
 		(at 157.48 92.71 0)
 		(unit 1)
@@
 			)
 		)
-		(property "Footprint" "nixie_clock:IN-12-DSUB"
+		(property "Footprint" "0_nixie_clock:IN-12-DSUB"
 			(at 158.242 88.9 0)
 			(effects
@@
 	)
 	(symbol
-		(lib_id "nixie_clock:IN-12B")
+		(lib_id "0_nixie_clock:IN-12B")
 		(at 74.93 44.45 0)
 		(unit 1)
@@
 			)
 		)
-		(property "Footprint" "nixie_clock:IN-12-DSUB"
+		(property "Footprint" "0_nixie_clock:IN-12-DSUB"
 			(at 75.692 40.64 0)
 			(effects
@@
 	)
 	(symbol
-		(lib_id "nixie_clock:IN-12B")
+		(lib_id "0_nixie_clock:IN-12B")
 		(at 157.48 43.18 0)
 		(unit 1)
@@
 			)
 		)
-		(property "Footprint" "nixie_clock:IN-12-DSUB"
+		(property "Footprint" "0_nixie_clock:IN-12-DSUB"
 			(at 158.242 39.37 0)
 			(effects
@@
 	)
 	(symbol
-		(lib_id "nixie_clock:IN-12B")
+		(lib_id "0_nixie_clock:IN-12B")
 		(at 74.93 93.98 0)
 		(unit 1)
@@
 			)
 		)
-		(property "Footprint" "nixie_clock:IN-12-DSUB"
+		(property "Footprint" "0_nixie_clock:IN-12-DSUB"
 			(at 75.692 90.17 0)
 			(effects
@@
 			)
 		)
-		(property "Footprint" "nixie_clock:C_Rect_L5.1mm_W3.2mm_P2.54mm_Goldmax"
+		(property "Footprint" "0_nixie_clock:C_Rect_L5.1mm_W3.2mm_P2.54mm_Goldmax"
 			(at 25.0952 86.36 0)
 			(effects
@@
 			)
 		)
-		(property "Footprint" "nixie_clock:C_Rect_L5.1mm_W3.2mm_P2.54mm_Goldmax"
+		(property "Footprint" "0_nixie_clock:C_Rect_L5.1mm_W3.2mm_P2.54mm_Goldmax"
 			(at 25.0952 36.83 0)
 			(effects
@@
 	)
 	(symbol
-		(lib_id "nixie_clock:K155ID1")
+		(lib_id "0_nixie_clock:K155ID1")
 		(at 129.54 90.17 0)
 		(unit 1)
@@
 			)
 		)
-		(property "Footprint" "nixie_clock:DIP16"
+		(property "Footprint" "0_nixie_clock:DIP16"
 			(at 130.302 86.36 0)
 			(effects
@@
 	)
 	(symbol
-		(lib_id "nixie_clock:K155ID1")
+		(lib_id "0_nixie_clock:K155ID1")
 		(at 129.54 40.64 0)
 		(unit 1)
@@
 			)
 		)
-		(property "Footprint" "nixie_clock:DIP16"
+		(property "Footprint" "0_nixie_clock:DIP16"
 			(at 130.302 36.83 0)
 			(effects
@@
 	)
 	(symbol
-		(lib_id "nixie_clock:IN-6")
+		(lib_id "0_nixie_clock:IN-6")
 		(at 204.47 36.83 0)
 		(unit 1)
@@
 			)
 		)
-		(property "Footprint" "nixie_clock:IN-6"
+		(property "Footprint" "0_nixie_clock:IN-6"
 			(at 205.232 33.02 0)
 			(effects

Commit message: Clock Face Rev C
Parts:
- removed C1, C3: 100nF, 0_nixie_clock:C_Rect_L5.1mm_W3.2mm_P2.54mm_Goldmax, symbol Device:C
- added C3: 47uF, 0_nixie_clock:CP_Radial_D6.3mm_P2.50mm, symbol Device:C_Polarized
- renumbered C2 to C1, C4 to C2, NX3 to NX1, NX6 to NX3, NX5 to NX4, NX1 to NX5, NX4 to NX6, R3 to R1, R6 to R3, R5 to R4, R1 to R5, R4 to R6, U2 to U1, U1 to U2, U4 to U3, U3 to U4
Connections:
- net +5V: now also C3.1
- net GND: now also C3.2
- net H10_{A}: now also J1.19 (Pin_19); no longer J1.23 (Pin_23)
- net H10_{B}: now also J1.23 (Pin_23); no longer J1.24 (Pin_24)
- net H10_{C}: now also J1.25 (Pin_25); no longer J1.26 (Pin_26)
- net H10_{D}: now also J1.21 (Pin_21); no longer J1.25 (Pin_25)
- net H1_{A}: now also J1.26 (Pin_26); no longer J1.21 (Pin_21)
- net H1_{B}: now also J1.22 (Pin_22); no longer J1.19 (Pin_19)
- net H1_{D}: now also J1.24 (Pin_24); no longer J1.22 (Pin_22)
- net M10_{B}: now also J1.4 (Pin_4); no longer J1.6 (Pin_6)
- net M10_{C}: now also J1.2 (Pin_2); no longer J1.5 (Pin_5)
- net M10_{D}: now also J1.6 (Pin_6); no longer J1.7 (Pin_7)
- net M1_{A}: now also J1.1 (Pin_1); no longer J1.2 (Pin_2)
- net M1_{B}: now also J1.5 (Pin_5); no longer J1.1 (Pin_1)
- net M1_{C}: now also J1.7 (Pin_7); no longer J1.3 (Pin_3)
- net M1_{D}: now also J1.3 (Pin_3); no longer J1.4 (Pin_4)
- net NX1_{0}: now also U1.11 (6); no longer U1.16 (0)
- net NX1_{1}: now also U1.13 (4); no longer U1.15 (1)
- net NX1_{2}: now also U1.14 (5); no longer U1.8 (2)
- net NX1_{3}: now also U1.15 (1); no longer U1.9 (3)
- net NX1_{4}: now also U1.16 (0); no longer U1.13 (4)
- net NX1_{5}: now also U1.2 (9); no longer U1.14 (5)
- net NX1_{6}: now also U1.1 (8); no longer U1.11 (6)
- net NX1_{7}: now also U1.8 (2); no longer U1.10 (7)
- net NX1_{8}: now also U1.9 (3); no longer U1.1 (8)
- net NX1_{9}: now also U1.10 (7); no longer U1.2 (9)
- net NX2_{0}: now also U2.11 (6); no longer U2.16 (0)
- net NX2_{1}: now also U2.13 (4); no longer U2.15 (1)
- net NX2_{2}: now also U2.14 (5); no longer U2.8 (2)
- net NX2_{3}: now also U2.15 (1); no longer U2.9 (3)
- net NX2_{4}: now also U2.16 (0); no longer U2.13 (4)
- net NX2_{5}: now also U2.2 (9); no longer U2.14 (5)
- net NX2_{6}: now also U2.1 (8); no longer U2.11 (6)
- net NX2_{7}: now also U2.8 (2); no longer U2.10 (7)
- net NX2_{8}: now also U2.9 (3); no longer U2.1 (8)
- net NX2_{9}: now also U2.10 (7); no longer U2.2 (9)
- net NX3_{0}: now also U3.11 (6); no longer U3.16 (0)
- net NX3_{1}: now also U3.13 (4); no longer U3.15 (1)
- net NX3_{2}: now also U3.14 (5); no longer U3.8 (2)
- net NX3_{3}: now also U3.15 (1); no longer U3.9 (3)
- net NX3_{4}: now also U3.16 (0); no longer U3.13 (4)
- net NX3_{5}: now also U3.2 (9); no longer U3.14 (5)
- net NX3_{6}: now also U3.1 (8); no longer U3.11 (6)
- net NX3_{7}: now also U3.8 (2); no longer U3.10 (7)
- net NX3_{8}: now also U3.9 (3); no longer U3.1 (8)
- net NX3_{9}: now also U3.10 (7); no longer U3.2 (9)
- net NX4_{0}: now also U4.11 (6); no longer U4.16 (0)
- net NX4_{1}: now also U4.13 (4); no longer U4.15 (1)
- net NX4_{2}: now also U4.14 (5); no longer U4.8 (2)
- net NX4_{3}: now also U4.15 (1); no longer U4.9 (3)
- net NX4_{4}: now also U4.16 (0); no longer U4.13 (4)
- net NX4_{5}: now also U4.2 (9); no longer U4.14 (5)
- net NX4_{6}: now also U4.1 (8); no longer U4.11 (6)
- net NX4_{7}: now also U4.8 (2); no longer U4.10 (7)
- net NX4_{8}: now also U4.9 (3); no longer U4.1 (8)
- net NX4_{9}: now also U4.10 (7); no longer U4.2 (9)
Other:
- note added: "Connector to HV Converter"
- note added: "Connector to MCU"
- moved on the sheet: C1, C2, H1, H2, H3, H4, J1, J2, NX1, NX2, NX3, NX4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

Commit message: Main board Rev C
Parts:
- removed NX5, NX6: IN-6, 0_nixie_clock:IN-6, symbol 0_nixie_clock:IN-6
- added NX5, NX6: INS-1, 0_nixie_clock:INS-1_Recessed, symbol 0_nixie_clock:INS-1
- C3: value 47uF -> 10uF; footprint 0_nixie_clock:CP_Radial_D6.3mm_P2.50mm -> Capacitor_THT:CP_Radial_D5.0mm_P2.00mm; MFG Part No A750EK476M1EAAE040 -> A758BG106M1EAAE070
Connections:
- net GND: now also NX5.K, NX6.K
- net NX5_{A}: now also NX5.A
- net NX6_{A}: now also NX6.A
Changed lines of the file:
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@@
 			)
 		)
-		(property "Value" "47uF"
+		(property "Value" "10uF"
 			(at 68.58 145.1609 0)
 			(show_name no)
@@
 			)
 		)
-		(property "Footprint" "0_nixie_clock:CP_Radial_D6.3mm_P2.50mm"
+		(property "Footprint" "Capacitor_THT:CP_Radial_D5.0mm_P2.00mm"
 			(at 65.7352 148.59 0)
 			(hide yes)
@@
 			)
 		)
-		(property "MFG Part No" "A750EK476M1EAAE040"
+		(property "MFG Part No" "A758BG106M1EAAE070"
 			(at 64.77 144.78 0)
 			(hide yes)
@@
 	)
 	(symbol
-		(lib_id "0_nixie_clock:IN-6")
-		(at 220.98 59.69 0)
-		(unit 1)
-		(body_style 1)
-		(exclude_from_sim no)
-		(in_bom no)
-		(on_board yes)
-		(in_pos_files yes)
-		(dnp no)
-		(fields_autoplaced yes)
-		(property "Reference" "NX6"
-			(at 220.98 52.07 0)
-			(show_name no)
-			(do_not_autoplace no)
-			(effects
-				(font
-					(size 1.143 1.143)
-				)
-			)
-		)
-		(property "Value" "IN-6"
-			(at 220.98 59.69 0)
-			(hide yes)
-			(show_name no)
-			(do_not_autoplace no)
-			(effects
-				(font
-					(size 1.143 1.143)
-				)
-				(justify left bottom)
-			)
-		)
-		(property "Footprint" "0_nixie_clock:IN-6"
-			(at 221.742 55.88 0)
-			(hide yes)
-			(show_name no)
-			(do_not_autoplace no)
-			(effects
-				(font
-					(size 0.508 0.508)
-				)
-			)
-		)
-		(property "Datasheet" ""
-			(at 220.98 59.69 0)
-			(hide yes)
-			(show_name no)
-			(do_not_autoplace no)
-			(effects
-				(font
-					(size 1.27 1.27)
-				)
-			)
-		)
-		(property "Description" "IN-6 neon dot indicator (colon separator); 3 electrodes: A=anode, K=indicator cathode, KA=auxiliary priming cathode (may be left NC in always-on use)"
-			(at 220.98 59.69 0)
-			(hide yes)
-			(show_name no)
-			(do_not_autoplace no)
-			(effects
-				(font
-					(size 1.27 1.27)
-				)
-			)
-		)
-		(property "MFG Part No" ""
-			(at 220.98 59.69 0)
-			(hide yes)
-			(show_name no)
-			(do_not_autoplace no)
-			(effects
-				(font
-					(size 1.27 1.27)
-				)
-			)
-		)
-		(property "LCSC" ""
-			(at 220.98 59.69 0)
-			(hide yes)
-			(show_name no)
-			(do_not_autoplace no)
-			(effects
-				(font
-					(size 1.27 1.27)
-				)
-			)
-		)
-		(pin "K"
-		)
-		(pin "A"
-		)
-		(pin "KA"
-		)
-		(instances
-			(project "face"
-				(path "/e9a806d6-34c6-4a58-8596-3336bf2feadc"
-					(reference "NX6")
-					(unit 1)
-				)
-			)
-		)
-	)
-	(symbol
 		(lib_id "0_nixie_clock:IN-12B")
 		(at 175.26 93.98 0)
@@
 	)
 	(symbol
+		(lib_id "0_nixie_clock:INS-1")
+		(at 220.98 59.69 0)
+		(unit 1)
+		(body_style 1)
+		(exclude_from_sim no)
+		(in_bom yes)
+		(on_board yes)
+		(in_pos_files yes)
+		(dnp no)
+		(fields_autoplaced yes)
+		(property "Reference" "NX6"
+			(at 220.98 49.53 0)
+			(show_name no)
+			(do_not_autoplace no)
+			(effects
+				(font
+					(size 1.143 1.143)
+				)
+			)
+		)
+		(property "Value" "INS-1"
+			(at 220.98 52.07 0)
+			(show_name no)
+			(do_not_autoplace no)
+			(effects
+				(font
+					(size 1.143 1.143)
+				)
+			)
+		)
+		(property "Footprint" "0_nixie_clock:INS-1_Recessed"
+			(at 221.742 55.88 0)
+			(hide yes)
+			(show_name no)
+			(do_not_autoplace no)
+			(effects
+				(font
+					(size 0.508 0.508)
+				)
+			)
+		)
+		(property "Datasheet" "${KIPRJMOD}/../../docs/datasheets/INS-1.pdf"
+			(at 220.98 59.69 0)
+			(hide yes)
+			(show_name no)
+			(do_not_autoplace no)
+			(effects
+				(font
+					(size 1.27 1.27)
+				)
+			)
+		)
+		(property "Description" "INS-1 neon glow indicator, colon separator; 2 electrodes, A = anode (small internal cylinder, lead 1), K = cathode (large cylinder, lead 2, the electrode the glow forms on). Strikes at 65 to 90 V, sustains at 55 V or less, 0.5 mA gives nominal brightness"
+			(at 220.98 59.69 0)
+			(hide yes)
+			(show_name no)
+			(do_not_autoplace no)
+			(effects
+				(font
+					(size 1.27 1.27)
+				)
+			)
+		)
+		(property "MFG Part No" ""
+			(at 220.98 59.69 0)
+			(hide yes)
+			(show_name no)
+			(do_not_autoplace no)
+			(effects
+				(font
+					(size 1.27 1.27)
+				)
+			)
+		)
+		(property "LCSC" ""
+			(at 220.98 59.69 0)
+			(hide yes)
+			(show_name no)
+			(do_not_autoplace no)
+			(effects
+				(font
+					(size 1.27 1.27)
+				)
+			)
+		)
+		(pin "A"
+		)
+		(pin "K"
+		)
+		(instances
+			(project "face"
+				(path "/e9a806d6-34c6-4a58-8596-3336bf2feadc"
+					(reference "NX6")
+					(unit 1)
+				)
+			)
+		)
+	)
+	(symbol
 		(lib_id "power:GND")
 		(at 231.14 62.23 0)
@@
 	)
 	(symbol
-		(lib_id "0_nixie_clock:IN-6")
-		(at 220.98 36.83 0)
+		(lib_id "power:+5V")
+		(at 111.76 86.36 0)
 		(unit 1)
 		(body_style 1)
 		(exclude_from_sim no)
-		(in_bom no)
+		(in_bom yes)
 		(on_board yes)
 		(in_pos_files yes)
 		(dnp no)
 		(fields_autoplaced yes)
-		(property "Reference" "NX5"
-			(at 220.98 29.21 0)
-			(show_name no)
-			(do_not_autoplace no)
-			(effects
-				(font
-					(size 1.143 1.143)
-				)
-			)
-		)
-		(property "Value" "IN-6"
-			(at 220.98 36.83 0)
-			(hide yes)
-			(show_name no)
-			(do_not_autoplace no)
-			(effects
-				(font
-					(size 1.143 1.143)
-				)
-				(justify left bottom)
-			)
-		)
-		(property "Footprint" "0_nixie_clock:IN-6"
-			(at 221.742 33.02 0)
+		(property "Reference" "#PWR07"
+			(at 111.76 90.17 0)
 			(hide yes)
 			(show_name no)
@@
 			(effects
 				(font
-					(size 0.508 0.508)
+					(size 1.27 1.27)
 				)
 			)
 		)
-		(property "Datasheet" ""
-			(at 220.98 36.83 0)
-			(hide yes)
+		(property "Value" "+5V"
+			(at 111.76 81.28 0)
 			(show_name no)
 			(do_not_autoplace no)
@@
 			)
 		)
-		(property "Description" "IN-6 neon dot indicator (colon separator); 3 electrodes: A=anode, K=indicator cathode, KA=auxiliary priming cathode (may be left NC in always-on use)"
-			(at 220.98 36.83 0)
+		(property "Footprint" ""
+			(at 111.76 86.36 0)
 			(hide yes)
 			(show_name no)
@@
 			)
 		)
-		(property "MFG Part No" ""
-			(at 220.98 36.83 0)
+		(property "Datasheet" ""
+			(at 111.76 86.36 0)
 			(hide yes)
 			(show_name no)
@@
 			)
 		)
-		(property "LCSC" ""
-			(at 220.98 36.83 0)
+		(property "Description" "Power symbol creates a global label with name \"+5V\""
+			(at 111.76 86.36 0)
 			(hide yes)
 			(show_name no)
@@
 			)
 		)
-		(pin "K"
-		)
-		(pin "A"
-		)
-		(pin "KA"
+		(pin "1"
 		)
 		(instances
 			(project "face"
 				(path "/e9a806d6-34c6-4a58-8596-3336bf2feadc"
-					(reference "NX5")
+					(reference "#PWR07")
 					(unit 1)
 				)
@@
 	)
 	(symbol
-		(lib_id "power:+5V")
-		(at 111.76 86.36 0)
+		(lib_id "0_nixie_clock:INS-1")
+		(at 220.98 36.83 0)
 		(unit 1)
 		(body_style 1)
@@
 		(dnp no)
 		(fields_autoplaced yes)
-		(property "Reference" "#PWR07"
-			(at 111.76 90.17 0)
+		(property "Reference" "NX5"
+			(at 220.98 26.67 0)
+			(show_name no)
+			(do_not_autoplace no)
+			(effects
+				(font
+					(size 1.143 1.143)
+				)
+			)
+		)
+		(property "Value" "INS-1"
+			(at 220.98 29.21 0)
+			(show_name no)
+			(do_not_autoplace no)
+			(effects
+				(font
+					(size 1.143 1.143)
+				)
+			)
+		)
+		(property "Footprint" "0_nixie_clock:INS-1_Recessed"
+			(at 221.742 33.02 0)
 			(hide yes)
 			(show_name no)
@@
 			(effects
 				(font
-					(size 1.27 1.27)
+					(size 0.508 0.508)
 				)
 			)
 		)
-		(property "Value" "+5V"
-			(at 111.76 81.28 0)
+		(property "Datasheet" "${KIPRJMOD}/../../docs/datasheets/INS-1.pdf"
+			(at 220.98 36.83 0)
+			(hide yes)
 			(show_name no)
 			(do_not_autoplace no)
@@
 			)
 		)
-		(property "Footprint" ""
-			(at 111.76 86.36 0)
+		(property "Description" "INS-1 neon glow indicator, colon separator; 2 electrodes, A = anode (small internal cylinder, lead 1), K = cathode (large cylinder, lead 2, the electrode the glow forms on). Strikes at 65 to 90 V, sustains at 55 V or less, 0.5 mA gives nominal brightness"
+			(at 220.98 36.83 0)
 			(hide yes)
 			(show_name no)
@@
 			)
 		)
-		(property "Datasheet" ""
-			(at 111.76 86.36 0)
+		(property "MFG Part No" ""
+			(at 220.98 36.83 0)
 			(hide yes)
 			(show_name no)
@@
 			)
 		)
-		(property "Description" "Power symbol creates a global label with name \"+5V\""
-			(at 111.76 86.36 0)
+		(property "LCSC" ""
+			(at 220.98 36.83 0)
 			(hide yes)
 			(show_name no)
@@
 			)
 		)
-		(pin "1"
+		(pin "A"
+		)
+		(pin "K"
 		)
 		(instances
 			(project "face"
 				(path "/e9a806d6-34c6-4a58-8596-3336bf2feadc"
-					(reference "#PWR07")
+					(reference "NX5")
 					(unit 1)
 				)

Commit message: Update release process, update analysis to use INS-1 throughout
Parts:
- R5, R6: value 120k -> 240k; MFG Part No MFR-25FRF52-120K -> CFR-25JR-52-240K
Changed lines of the file:
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@@
 			)
 		)
-		(property "Value" "120k"
+		(property "Value" "240k"
 			(at 210.82 54.6099 0)
 			(show_name no)
@@
 			)
 		)
-		(property "MFG Part No" "MFR-25FRF52-120K"
+		(property "MFG Part No" "CFR-25JR-52-240K"
+			(at 208.28 53.34 0)
+			(hide yes)
+			(show_name no)
+			(do_not_autoplace no)
+			(effects
+				(font
+					(size 1.27 1.27)
+				)
+			)
+		)
+		(property "LCSC" ""
 			(at 208.28 53.34 0)
 			(hide yes)
@@
 			)
 		)
-		(property "Value" "120k"
+		(property "Value" "240k"
 			(at 210.82 31.7499 0)
 			(show_name no)
@@
 			)
 		)
-		(property "MFG Part No" "MFR-25FRF52-120K"
+		(property "MFG Part No" "CFR-25JR-52-240K"
 			(at 208.28 30.48 0)
 			(hide yes)

Commit message: Update face schematic footprints
Parts:
- NX5, NX6: footprint 0_nixie_clock:INS-1_Recessed -> 0_nixie_clock:INS-1
Changed lines of the file:
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@@
 			)
 		)
-		(property "Footprint" "0_nixie_clock:INS-1_Recessed"
+		(property "Footprint" "0_nixie_clock:INS-1"
 			(at 221.742 55.88 0)
 			(hide yes)
@@
 			)
 		)
-		(property "Footprint" "0_nixie_clock:INS-1_Recessed"
+		(property "Footprint" "0_nixie_clock:INS-1"
 			(at 221.742 33.02 0)
 			(hide yes)
