File: pcb/face/face.kicad_sch (KiCad schematic)
At the start: 25 parts, among them J1 26 pin IDC, J2 Phoenix MSTB, U1 K155ID1, U2 K155ID1, U3 K155ID1, U4 K155ID1

Commit message: Fix ballast/divider resistors to match first line of table 5-2
Parts:
- R1, R2, R3, R4: value 8.2k -> 7.5k; MFG Part No MFR-25FTE52-8K2 -> MFR-25FTE52-7K5
Changed lines of the file:
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@@
 			)
 		)
-		(property "Value" "8.2k"
+		(property "Value" "7.5k"
 			(at 193.04 38.0999 0)
 			(show_name no)
@@
 			)
 		)
-		(property "MFG Part No" "MFR-25FTE52-8K2"
+		(property "MFG Part No" "MFR-25FTE52-7K5"
 			(at 190.5 36.83 0)
 			(hide yes)
@@
 			)
 		)
-		(property "Value" "8.2k"
+		(property "Value" "7.5k"
 			(at 104.14 39.3699 0)
 			(show_name no)
@@
 			)
 		)
-		(property "MFG Part No" "MFR-25FTE52-8K2"
+		(property "MFG Part No" "MFR-25FTE52-7K5"
 			(at 101.6 38.1 0)
 			(hide yes)
@@
 			)
 		)
-		(property "Value" "8.2k"
+		(property "Value" "7.5k"
 			(at 193.04 88.8999 0)
 			(show_name no)
@@
 			)
 		)
-		(property "MFG Part No" "MFR-25FTE52-8K2"
+		(property "MFG Part No" "MFR-25FTE52-7K5"
 			(at 190.5 87.63 0)
 			(hide yes)
@@
 			)
 		)
-		(property "Value" "8.2k"
+		(property "Value" "7.5k"
 			(at 104.14 88.8999 0)
 			(show_name no)
@@
 			)
 		)
-		(property "MFG Part No" "MFR-25FTE52-8K2"
+		(property "MFG Part No" "MFR-25FTE52-7K5"
 			(at 101.6 87.63 0)
 			(hide yes)

Commit message: Update ins1 tube model, update hv/main connector to 1 vbus, 2 gnd connections, update hv inhibit circuit to be default inhibit and require positive enable from MCU
Parts:
- J1: MFG Part No (none) -> 75869-105LF; Note (none) -> Mates with 71600-026LF; now in the parts list
- J2: MFG Part No 1757255 -> 1755749; now in the parts list
- NX5, NX6: footprint 0_nixie_clock:INS-1 -> 0_nixie_clock:INS-1_Recessed
Connections:
- net GND: now also J1.10 (Pin_10), J1.17 (Pin_17), J1.18 (Pin_18), J1.9 (Pin_9)
- no-connect marks 11 -> 7
Changed lines of the file:
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@@
 	)
 	(junction
+		(at 22.86 148.59)
+		(diameter 0)
+		(color 0 0 0 0)
+	)
+	(junction
 		(at 22.86 143.51)
 		(diameter 0)
@@
 	)
 	(junction
+		(at 50.8 148.59)
+		(diameter 0)
+		(color 0 0 0 0)
+	)
+	(junction
 		(at 22.86 146.05)
 		(diameter 0)
@@
 	)
 	(junction
+		(at 64.77 148.59)
+		(diameter 0)
+		(color 0 0 0 0)
+	)
+	(junction
 		(at 83.82 134.62)
 		(diameter 0)
@@
 		(color 0 0 0 0)
 	)
-	(no_connect
-		(at 96.52 81.28)
-	)
-	(no_connect
-		(at 48.26 138.43)
+	(junction
+		(at 22.86 140.97)
+		(diameter 0)
+		(color 0 0 0 0)
 	)
 	(no_connect
-		(at 48.26 148.59)
+		(at 96.52 81.28)
 	)
 	(no_connect
@@
 	)
 	(no_connect
-		(at 35.56 138.43)
-	)
-	(no_connect
 		(at 185.42 30.48)
 	)
 	(no_connect
-		(at 35.56 148.59)
-	)
-	(no_connect
 		(at 83.82 132.08)
 	)
 	(wire
 		(pts
+			(xy 35.56 138.43) (xy 22.86 138.43)
+		)
+		(stroke
+			(width 0)
+			(type default)
+		)
+	)
+	(wire
+		(pts
+			(xy 22.86 148.59) (xy 35.56 148.59)
+		)
+		(stroke
+			(width 0)
+			(type default)
+		)
+	)
+	(wire
+		(pts
+			(xy 48.26 138.43) (xy 50.8 138.43)
+		)
+		(stroke
+			(width 0)
+			(type default)
+		)
+	)
+	(wire
+		(pts
 			(xy 48.26 143.51) (xy 59.69 143.51)
 		)
@@
 	(wire
 		(pts
+			(xy 50.8 148.59) (xy 64.77 148.59)
+		)
+		(stroke
+			(width 0)
+			(type default)
+		)
+	)
+	(wire
+		(pts
 			(xy 59.69 138.43) (xy 59.69 140.97)
 		)
@@
 	(wire
 		(pts
+			(xy 48.26 148.59) (xy 50.8 148.59)
+		)
+		(stroke
+			(width 0)
+			(type default)
+		)
+	)
+	(wire
+		(pts
 			(xy 111.76 88.9) (xy 121.92 88.9)
 		)
@@
 	(wire
 		(pts
-			(xy 22.86 149.86) (xy 22.86 146.05)
+			(xy 22.86 149.86) (xy 22.86 148.59)
 		)
 		(stroke
@@
 	(wire
 		(pts
+			(xy 22.86 148.59) (xy 22.86 146.05)
+		)
+		(stroke
+			(width 0)
+			(type default)
+		)
+	)
+	(wire
+		(pts
 			(xy 24.13 88.9) (xy 34.29 88.9)
 		)
@@
 	(wire
 		(pts
+			(xy 50.8 138.43) (xy 50.8 148.59)
+		)
+		(stroke
+			(width 0)
+			(type default)
+		)
+	)
+	(wire
+		(pts
 			(xy 62.23 138.43) (xy 62.23 140.97)
 		)
@@
 	(wire
 		(pts
+			(xy 22.86 138.43) (xy 22.86 140.97)
+		)
+		(stroke
+			(width 0)
+			(type default)
+		)
+	)
+	(wire
+		(pts
 			(xy 62.23 140.97) (xy 64.77 140.97)
 		)
@@
 			)
 		)
-		(property "Footprint" "0_nixie_clock:INS-1"
+		(property "Footprint" "0_nixie_clock:INS-1_Recessed"
 			(at 221.742 55.88 0)
 			(hide yes)
@@
 		(body_style 1)
 		(exclude_from_sim no)
-		(in_bom no)
+		(in_bom yes)
 		(on_board yes)
 		(in_pos_files yes)
@@
 			)
 		)
-		(property "MFG Part No" "1757255"
+		(property "MFG Part No" "1755749"
 			(at 88.9 132.08 0)
 			(hide yes)
@@
 		(body_style 1)
 		(exclude_from_sim no)
-		(in_bom no)
+		(in_bom yes)
 		(on_board yes)
 		(in_pos_files yes)
@@
 			)
 		)
-		(property "MFG Part No" ""
+		(property "MFG Part No" "75869-105LF"
 			(at 40.64 143.51 0)
 			(hide yes)
@@
 			)
 		)
+		(property "Note" "Mates with 71600-026LF"
+			(at 40.64 143.51 0)
+			(hide yes)
+			(show_name no)
+			(do_not_autoplace no)
+			(effects
+				(font
+					(size 1.27 1.27)
+				)
+			)
+		)
 		(pin "9"
 		)
@@
 			)
 		)
-		(property "Footprint" "0_nixie_clock:INS-1"
+		(property "Footprint" "0_nixie_clock:INS-1_Recessed"
 			(at 221.742 33.02 0)
 			(hide yes)
