File: pcb/face/face.kicad_sch (KiCad schematic)
At the start: 25 parts, among them J1 26 pin IDC, J2 Phoenix MSTB, U1 K155ID1, U2 K155ID1, U3 K155ID1, U4 K155ID1

Commit message: Update face to Rev D, update IN-12 footprint to accomodate properly sized pin sockets.
Parts:
- NX1, NX2, NX3, NX4: Note (none) -> Individual 0327-0-15-15-34-27-10-0 sockets for pins
Changed lines of the file:
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@@
+			)
+		)
+		(property "Note" "Individual 0327-0-15-15-34-27-10-0 sockets for pins"
+			(at 175.26 93.98 0)
+			(hide yes)
+			(show_name no)
+			(do_not_autoplace no)
+			(effects
+				(font
+					(size 1.27 1.27)
+				)
 			)
 		)
@@
 			)
 		)
+		(property "Note" "Individual 0327-0-15-15-34-27-10-0 sockets for pins"
+			(at 86.36 44.45 0)
+			(hide yes)
+			(show_name no)
+			(do_not_autoplace no)
+			(effects
+				(font
+					(size 1.27 1.27)
+				)
+			)
+		)
 		(pin "4"
 		)
@@
 			)
 		)
+		(property "Note" "Individual 0327-0-15-15-34-27-10-0 sockets for pins"
+			(at 175.26 43.18 0)
+			(hide yes)
+			(show_name no)
+			(do_not_autoplace no)
+			(effects
+				(font
+					(size 1.27 1.27)
+				)
+			)
+		)
 		(pin "4"
 		)
@@
 			(at 86.36 93.98 0)
 			(hide yes)
+			(show_name no)
+			(do_not_autoplace no)
+			(effects
+				(font
+					(size 1.27 1.27)
+				)
+			)
+		)
+		(property "Note" "Individual 0327-0-15-15-34-27-10-0 sockets for pins"
+			(at 86.36 93.98 0)
+			(hide yes)
