File: pcb/hv/hv.kicad_sch (KiCad schematic)
At the start: 51 parts, among them J1 JST XH, J2 Phoenix MSTB, Q1 IRL540N, Q2 TN2106N3-G, Q3 TN2106N3-G, T1 DA2032-AL, U1 LM5156H

Commit message: Change C9 to 2.2uF, slows slow start to ~200ms
Parts:
- C9: value 470nF -> 2.2uF; MFG Part No C322C474K5R5TA7301 -> C322C225K5R5TA
Changed lines of the file:
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@@
 			)
 		)
-		(property "Value" "470nF"
+		(property "Value" "2.2uF"
 			(at 91.44 95.2499 0)
 			(show_name no)
@@
 			)
 		)
-		(property "MFG Part No" "C322C474K5R5TA7301"
+		(property "MFG Part No" "C322C225K5R5TA"
 			(at 87.63 93.98 0)
 			(hide yes)
